File: kicad/controller.sch (KiCad schematic (older format))
At the start: 4 parts

Commit message: Pulled all into one schematic - don't know yet if this is a good idea.
Parts:
- removed Q?: MPSA92, Package_TO_SOT_THT:TO-92_Inline, symbol Transistor_BJT:MPSA92
- R?: footprint (none) -> Resistor_SMD:R_0805_2012Metric_Pad1.15x1.40mm_HandSolder
Changed lines of the file:
@@
 EESchema Schematic File Version 4
+LIBS:funknetzwerkuhr-cache
 LIBS:nixie-breakout-cache
 EELAYER 26 0
@@
 $Descr A4 11693 8268
 encoding utf-8
-Sheet 2 2
+Sheet 2 4
 Title ""
 Date ""
@@
 Comment4 ""
 $EndDescr
-$Comp
-L Transistor_BJT:MPSA92 Q?
-U 1 1 5B3B9AF7
-P 5550 5500
-F 0 "Q?" H 5741 5546 50  0000 L CNN
-F 1 "MPSA92" H 5741 5455 50  0000 L CNN
-F 2 "Package_TO_SOT_THT:TO-92_Inline" H 5750 5425 50  0001 L CIN
-F 3 "http://www.onsemi.com/pub_link/Collateral/MPSA92-D.PDF" H 5550 5500 50  0001 L CNN
-	1    5550 5500
-	1    0    0    -1
-$EndComp
 $Comp
 L Transistor_BJT:MPSA92 Q?
@@
 F 0 "R?" H 1670 1896 50  0000 L CNN
 F 1 "R" H 1670 1805 50  0000 L CNN
-F 2 "" V 1530 1850 50  0001 C CNN
+F 2 "Resistor_SMD:R_0805_2012Metric_Pad1.15x1.40mm_HandSolder" V 1530 1850 50  0001 C CNN
 F 3 "~" H 1600 1850 50  0001 C CNN
 	1    1600 1850
