File: kicad/front_panel.sch (KiCad schematic (older format))
At the start: 11 parts

Commit message: Schematic nearly done, need to add programming header.
Parts:
- added J3: Conn_01x26_Female, Connector_PinSocket_2.54mm:PinSocket_1x26_P2.54mm_Vertical, symbol Connector:Conn_01x26_Female
- gave numbers to parts that had none: 11
Connections:
- net labels added: A1, A2, A3, A4, ANODE_1, ANODE_2, ANODE_3, ANODE_4, D0, D1, D2, D3, D4, D5, D6, D7, D8, D9, DIGIT_0, DIGIT_1, DIGIT_2, DIGIT_3, DIGIT_4, DIGIT_5, DIGIT_6, DIGIT_7, DIGIT_8, DIGIT_9, DIGIT_DOT, DOT
- wire segments 175 -> 206

Commit message: Schematic complete. PCB nearly done.
Connections:
- net labels added: ANODE_LED_1, ANODE_LED_2, ANODE_LED_3, ANODE_LED_4, ANODE_N1, ANODE_N2, BLUE, CATHODE_N1, CATHODE_N2, GREEN, RED
Changed lines of the file:
@@
 $Descr A4 11693 8268
 encoding utf-8
-Sheet 3 3
+Sheet 2 3
 Title ""
 Date ""
@@
 Text Label 2650 3850 0    50   ~ 0
 D6
+Text HLabel 1700 3950 0    50   Input ~ 0
+ANODE_N1
+Text HLabel 1700 4050 0    50   Input ~ 0
+CATHODE_N1
+Text HLabel 1700 4150 0    50   Input ~ 0
+ANODE_N2
+Text HLabel 1700 4250 0    50   Input ~ 0
+CATHODE_N2
+Text HLabel 1700 4350 0    50   Input ~ 0
+RED
+Text HLabel 1700 4450 0    50   Input ~ 0
+GREEN
+Text HLabel 1700 4550 0    50   Input ~ 0
+BLUE
+Text HLabel 1700 4650 0    50   Input ~ 0
+ANODE_LED_1
+Text HLabel 1700 4750 0    50   Input ~ 0
+ANODE_LED_2
+Text HLabel 1700 4850 0    50   Input ~ 0
+ANODE_LED_3
+Text HLabel 1700 4950 0    50   Input ~ 0
+ANODE_LED_4
 $EndSCHEMATC
