File: kicad/funknetzwerkuhr.kicad_pcb (KiCad board)
At the start: 2 copper layers, 80 x 130 mm, 11 parts, among them J1 Conn_01x26_Male, T1 IN-12, T2 IN-12, T3 IN-12, T4 IN-12

Commit message: Pulled all into one schematic - don't know yet if this is a good idea.
Parts:
- added C1: 10uF,25V, Capacitor_THT:CP_Radial_D5.0mm_P2.50mm, F.Cu at (200.1, 148.6)
- added C2: 100n, Capacitor_SMD:C_1206_3216Metric_Pad1.42x1.75mm_HandSolder, F.Cu at (178.1, 149.8)
- added C3: 100n, Capacitor_SMD:C_1206_3216Metric_Pad1.42x1.75mm_HandSolder, F.Cu at (213.7, 127.2)
- added C4: 100uF,25V, Capacitor_THT:CP_Radial_D8.0mm_P3.50mm, F.Cu at (209.9, 141.5)
- added C5: 4.7uF,250V, Capacitor_THT:CP_Radial_D8.0mm_P3.50mm, F.Cu at (201.2, 141.5)
- added C6: 100p 1kV, Capacitor_THT:C_Disc_D4.3mm_W1.9mm_P5.00mm, F.Cu at (176.7, 147.4)
- added C7: 100n,250V, Capacitor_THT:C_Rect_L26.5mm_W5.0mm_P22.50mm_MKS4, F.Cu at (169.9, 128.8)
- added D5: LED_RGB_CA, Parts:LED_3528_3.5x2.8mm, F.Cu at (195.2, 95.9)
- added J2: Conn_01x26_Male, Connector_PinSocket_2.54mm:PinSocket_1x26_P2.54mm_Vertical, F.Cu at (124.9, 132.1)
- added L3: ins-1, Parts:ins-1, F.Cu at (182.4, 97.6)
- added Q1: IRF640, Package_TO_SOT_SMD:TO-263-2, F.Cu at (176.0, 137.3)
- added Q2: MPSA42, Package_TO_SOT_THT:TO-92_Inline, F.Cu at (319.3, 55.6)
- added Q3: MPSA92, Package_TO_SOT_THT:TO-92_Inline, F.Cu at (305.8, 66.1)
- added R1: 1.5M, Resistor_SMD:R_1206_3216Metric_Pad1.42x1.75mm_HandSolder, F.Cu at (178.1, 152.1)
- added R1a1: 2.7k, Resistor_SMD:R_0805_2012Metric_Pad1.15x1.40mm_HandSolder, F.Cu at (169.5, 152.6)
- added R2: 10k, Resistor_SMD:R_0805_2012Metric_Pad1.15x1.40mm_HandSolder, F.Cu at (173.3, 152.6)
- added R3: R, Resistor_SMD:R_0805_2012Metric_Pad1.15x1.40mm_HandSolder, F.Cu at (306.2, 69.1)
- added R4: 100k, Resistor_SMD:R_0805_2012Metric_Pad1.15x1.40mm_HandSolder, F.Cu at (311.7, 64.4)
- added RSENSE1: 0R1, Resistor_THT:R_Axial_DIN0516_L15.5mm_D5.0mm_P5.08mm_Vertical, F.Cu at (187.1, 134.4)
- added U1: 74HC595, Package_SO:SOIC-16_3.9x9.9mm_P1.27mm, F.Cu at (299.2, 58.1)
- added U2: 74HC595, Package_SO:SOIC-16_3.9x9.9mm_P1.27mm, F.Cu at (306.6, 58.1)
- added U3: 74HC595, Package_SO:SOIC-16_3.9x9.9mm_P1.27mm, F.Cu at (314.1, 58.1)
- added U4: max1771, Package_SO:PowerIntegrations_SO-8, F.Cu at (171.6, 148.9)
- added U5: AP1117-33, Package_TO_SOT_SMD:SOT-223-3_TabPin2, F.Cu at (299.9, 67.0)
- D1: value LED_RGB_CA -> ES2J; footprint Parts:LED_3528_3.5x2.8mm -> Parts:D_MELF-RM10_Universal_Handsoldering
- D2, D3: footprint Parts:LED_3528_3.5x2.8mm -> PartsStash:LED_3528_3.5x2.8mm
- J1: value Conn_01x26_Male -> Jack-DC; footprint Connector_PinSocket_2.54mm:PinSocket_1x26_P2.54mm_Vertical -> Parts:AliExpress55mmBarelJack
- L1: value ins-1 -> L; footprint Parts:ins-1 -> Inductor_THT:L_Toroid_Vertical_L16.0mm_W8.0mm_P7.62mm
- moved T2 152.1 mm to (226.6, 73.4), turned to 0 degrees
- moved L1 128.9 mm to (203.0, 127.8), turned to 0 degrees
- moved T3 123.1 mm to (204.5, 73.4), turned to 0 degrees
- moved D4 113.4 mm to (189.2, 95.9), turned to 0 degrees
- moved D3 108.9 mm to (189.2, 100.0), turned to 0 degrees
- moved T4 101.6 mm to (182.3, 73.4), turned to 0 degrees
- moved D2 94.0 mm to (174.3, 103.4), turned to 0 degrees
- moved D1 92.4 mm to (174.1, 144.6), turned to 0 degrees
- moved L2 86.7 mm to (175.0, 97.6), turned to 0 degrees
- moved J1 65.7 mm to (189.4, 144.7), turned to 0 degrees
Connections:
- D1 pad 1: Net-(D1-Pad1) -> +VDC
- D2 pad 1: Net-(D1-Pad1) -> Net-(D2-Pad1)
- D2 pad 3: Net-(D1-Pad3) -> Net-(D2-Pad3)
- D2 pad 4: Net-(D1-Pad4) -> Net-(D2-Pad4)
- D3 pad 1: Net-(D1-Pad1) -> Net-(D2-Pad1)
- D3 pad 3: Net-(D1-Pad3) -> Net-(D2-Pad3)
- D3 pad 4: Net-(D1-Pad4) -> Net-(D2-Pad4)
- D4 pad 1: Net-(D1-Pad1) -> Net-(D2-Pad1)
- D4 pad 3: Net-(D1-Pad3) -> Net-(D2-Pad3)
- D4 pad 4: Net-(D1-Pad4) -> Net-(D2-Pad4)
- J1 pad 1: Net-(J1-Pad1) -> +9V
- J1 pad 2: Net-(J1-Pad2) -> GND
- J1 pad 3: Net-(J1-Pad3) -> GND
- L1 pad 1: Net-(J1-Pad16) -> +9V
- L1 pad 2: Net-(J1-Pad17) -> Net-(D1-Pad2)
- L2 pad 1: Net-(J1-Pad18) -> Net-(J2-Pad16)
- L2 pad 2: Net-(J1-Pad19) -> Net-(J2-Pad17)
- T1 pad 1: Net-(J1-Pad1) -> Net-(J2-Pad1)
- T1 pad 10: Net-(J1-Pad5) -> Net-(J2-Pad5)
- T1 pad 11: Net-(J1-Pad6) -> Net-(J2-Pad6)
- T1 pad 12: Net-(J1-Pad15) -> Net-(J2-Pad15)
- T1 pad 2: Net-(J1-Pad7) -> Net-(J2-Pad7)
- T1 pad 3: Net-(J1-Pad14) -> Net-(J2-Pad14)
- T1 pad 4: Net-(J1-Pad13) -> Net-(J2-Pad13)
- T1 pad 5: Net-(J1-Pad12) -> Net-(J2-Pad12)
- T1 pad 6: Net-(J1-Pad11) -> Net-(J2-Pad11)
- T1 pad 7: Net-(J1-Pad10) -> Net-(J2-Pad10)
- T1 pad 8: Net-(J1-Pad9) -> Net-(J2-Pad9)
- T1 pad 9: Net-(J1-Pad8) -> Net-(J2-Pad8)
- T2 pad 1: Net-(J1-Pad2) -> Net-(J2-Pad2)
- T2 pad 10: Net-(J1-Pad5) -> Net-(J2-Pad5)
- T2 pad 11: Net-(J1-Pad6) -> Net-(J2-Pad6)
- T2 pad 12: Net-(J1-Pad15) -> Net-(J2-Pad15)
- T2 pad 2: Net-(J1-Pad7) -> Net-(J2-Pad7)
- T2 pad 3: Net-(J1-Pad14) -> Net-(J2-Pad14)
- T2 pad 4: Net-(J1-Pad13) -> Net-(J2-Pad13)
- T2 pad 5: Net-(J1-Pad12) -> Net-(J2-Pad12)
- T2 pad 6: Net-(J1-Pad11) -> Net-(J2-Pad11)
- T2 pad 7: Net-(J1-Pad10) -> Net-(J2-Pad10)
- T2 pad 8: Net-(J1-Pad9) -> Net-(J2-Pad9)
- T2 pad 9: Net-(J1-Pad8) -> Net-(J2-Pad8)
- T3 pad 1: Net-(J1-Pad3) -> Net-(J2-Pad3)
- T3 pad 10: Net-(J1-Pad5) -> Net-(J2-Pad5)
- T3 pad 11: Net-(J1-Pad6) -> Net-(J2-Pad6)
- T3 pad 12: Net-(J1-Pad15) -> Net-(J2-Pad15)
- T3 pad 2: Net-(J1-Pad7) -> Net-(J2-Pad7)
- T3 pad 3: Net-(J1-Pad14) -> Net-(J2-Pad14)
- T3 pad 4: Net-(J1-Pad13) -> Net-(J2-Pad13)
- T3 pad 5: Net-(J1-Pad12) -> Net-(J2-Pad12)
- T3 pad 6: Net-(J1-Pad11) -> Net-(J2-Pad11)
- T3 pad 7: Net-(J1-Pad10) -> Net-(J2-Pad10)
- T3 pad 8: Net-(J1-Pad9) -> Net-(J2-Pad9)
- T3 pad 9: Net-(J1-Pad8) -> Net-(J2-Pad8)
- T4 pad 1: Net-(J1-Pad4) -> Net-(J2-Pad4)
- T4 pad 10: Net-(J1-Pad5) -> Net-(J2-Pad5)
- T4 pad 11: Net-(J1-Pad6) -> Net-(J2-Pad6)
- T4 pad 12: Net-(J1-Pad15) -> Net-(J2-Pad15)
- T4 pad 2: Net-(J1-Pad7) -> Net-(J2-Pad7)
- T4 pad 3: Net-(J1-Pad14) -> Net-(J2-Pad14)
- T4 pad 4: Net-(J1-Pad13) -> Net-(J2-Pad13)
- T4 pad 5: Net-(J1-Pad12) -> Net-(J2-Pad12)
- T4 pad 6: Net-(J1-Pad11) -> Net-(J2-Pad11)
- T4 pad 7: Net-(J1-Pad10) -> Net-(J2-Pad10)
- T4 pad 8: Net-(J1-Pad9) -> Net-(J2-Pad9)
- T4 pad 9: Net-(J1-Pad8) -> Net-(J2-Pad8)
Routing:
- net Net-(D2-Pad3): track 0.00 -> 234.1 mm, vias 0 -> 9
- net Net-(D1-Pad3): track 234.1 -> 0.00 mm, vias 9 -> 0
- net Net-(J2-Pad15): track 0.00 -> 230.7 mm, vias 0 -> 6
- net Net-(J1-Pad15): track 230.7 -> 0.00 mm, vias 6 -> 0
- net Net-(J2-Pad14): track 0.00 -> 210.7 mm, vias 0 -> 5
- net Net-(J1-Pad14): track 210.7 -> 0.00 mm, vias 5 -> 0
- net Net-(J2-Pad7): track 0.00 -> 198.9 mm, vias 0 -> 5
- net Net-(J1-Pad7): track 198.9 -> 0.00 mm, vias 5 -> 0
- net Net-(J2-Pad6): track 0.00 -> 191.3 mm, vias 0 -> 5
- net Net-(J1-Pad6): track 191.3 -> 0.00 mm, vias 5 -> 0
- net Net-(J2-Pad5): track 0.00 -> 189.5 mm, vias 0 -> 5
- net Net-(J1-Pad5): track 189.5 -> 0.00 mm, vias 5 -> 0
- net Net-(D2-Pad1): track 0.00 -> 179.5 mm, vias 0 -> 2
- net Net-(D1-Pad1): track 179.5 -> 0.00 mm, vias 2 -> 0
- net Net-(J2-Pad8): track 0.00 -> 173.3 mm, vias 0 -> 6
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
Commit message: Schematic nearly done, need to add programming header.
Parts:
- removed C1: 10uF,25V, Capacitor_THT:CP_Radial_D5.0mm_P2.50mm
- added J3: Conn_01x26_Female, Connector_PinSocket_2.54mm:PinSocket_1x26_P2.54mm_Vertical, F.Cu at (215.7, 130.2)
- added Q10: MMBTA42, Package_TO_SOT_SMD:SOT-323_SC-70_Handsoldering, F.Cu at (208.9, 97.2)
- added Q11: MMBTA42, Package_TO_SOT_SMD:SOT-323_SC-70_Handsoldering, F.Cu at (208.9, 108.6)
- added Q12: MMBTA42, Package_TO_SOT_SMD:SOT-323_SC-70_Handsoldering, F.Cu at (208.9, 112.4)
- added Q13: MMBTA42, Package_TO_SOT_SMD:SOT-323_SC-70_Handsoldering, B.Cu at (209.0, 108.6)
- added Q14: MMBTA42, Package_TO_SOT_SMD:SOT-323_SC-70_Handsoldering, B.Cu at (208.9, 120.0)
- added Q15: MMBTA42, Package_TO_SOT_SMD:SOT-323_SC-70_Handsoldering, B.Cu at (208.9, 116.2)
- added Q16: MMBTA42, Package_TO_SOT_SMD:SOT-323_SC-70_Handsoldering, B.Cu at (208.9, 93.3)
- added Q17: MMBTA42, Package_TO_SOT_SMD:SOT-323_SC-70_Handsoldering, F.Cu at (208.9, 101.0)
- added Q18: MMBTA42, Package_TO_SOT_SMD:SOT-323_SC-70_Handsoldering, B.Cu at (209.0, 112.4)
- added Q19: MMBTA42, Package_TO_SOT_SMD:SOT-323_SC-70_Handsoldering, F.Cu at (208.9, 93.3)
- added Q20: MMBTA42, Package_TO_SOT_SMD:SOT-323_SC-70_Handsoldering, F.Cu at (208.9, 104.8)
- added Q4: MMBTA42, Package_TO_SOT_SMD:SOT-323_SC-70_Handsoldering, F.Cu at (188.8, 127.5)
- added Q5: MMBTA92, Package_TO_SOT_SMD:SOT-323_SC-70_Handsoldering, F.Cu at (200.3, 127.5)
- added Q6: MMBTA42, Package_TO_SOT_SMD:SOT-323_SC-70_Handsoldering, B.Cu at (188.8, 125.0)
- added Q7: MMBTA92, Package_TO_SOT_SMD:SOT-323_SC-70_Handsoldering, B.Cu at (200.2, 125.0)
- added Q8: MMBTA42, Package_TO_SOT_SMD:SOT-323_SC-70_Handsoldering, F.Cu at (188.8, 123.8)
- added Q9: MMBTA92, Package_TO_SOT_SMD:SOT-323_SC-70_Handsoldering, F.Cu at (200.2, 122.4)
- added R10: 1M, Resistor_SMD:R_0805_2012Metric_Pad1.15x1.40mm_HandSolder, F.Cu at (193.3, 127.5)
- added R11: 8k, Resistor_SMD:R_0805_2012Metric_Pad1.15x1.40mm_HandSolder, F.Cu at (205.2, 127.6)
- added R12: 33k, Resistor_SMD:R_0805_2012Metric_Pad1.15x1.40mm_HandSolder, B.Cu at (184.4, 125.0)
- added R13: 1M, Resistor_SMD:R_0805_2012Metric_Pad1.15x1.40mm_HandSolder, B.Cu at (195.8, 125.0)
- added R14: 1M, Resistor_SMD:R_0805_2012Metric_Pad1.15x1.40mm_HandSolder, B.Cu at (193.3, 125.0)
- added R15: 8k, Resistor_SMD:R_0805_2012Metric_Pad1.15x1.40mm_HandSolder, B.Cu at (205.3, 125.1)
- added R16: 33k, Resistor_SMD:R_0805_2012Metric_Pad1.15x1.40mm_HandSolder, F.Cu at (188.6, 119.4)
- added R17: 1M, Resistor_SMD:R_0805_2012Metric_Pad1.15x1.40mm_HandSolder, F.Cu at (195.8, 122.4)
- added R18: 1M, Resistor_SMD:R_0805_2012Metric_Pad1.15x1.40mm_HandSolder, F.Cu at (193.3, 122.4)
- added R19: 8k, Resistor_SMD:R_0805_2012Metric_Pad1.15x1.40mm_HandSolder, F.Cu at (205.3, 122.6)
- added R20: 33k, Resistor_SMD:R_0805_2012Metric_Pad1.15x1.40mm_HandSolder, F.Cu at (203.8, 96.5)
- added R21: 33k, Resistor_SMD:R_0805_2012Metric_Pad1.15x1.40mm_HandSolder, F.Cu at (203.8, 108.0)
- added R22: 33k, Resistor_SMD:R_0805_2012Metric_Pad1.15x1.40mm_HandSolder, F.Cu at (203.8, 111.8)
- added R23: 33k, Resistor_SMD:R_0805_2012Metric_Pad1.15x1.40mm_HandSolder, B.Cu at (203.8, 109.2)
- added R24: 33k, Resistor_SMD:R_0805_2012Metric_Pad1.15x1.40mm_HandSolder, B.Cu at (203.8, 120.7)
- added R25: 33k, Resistor_SMD:R_0805_2012Metric_Pad1.15x1.40mm_HandSolder, B.Cu at (203.8, 116.8)
- added R26: 33k, Resistor_SMD:R_0805_2012Metric_Pad1.15x1.40mm_HandSolder, B.Cu at (203.8, 94.0)
- added R27: 33k, Resistor_SMD:R_0805_2012Metric_Pad1.15x1.40mm_HandSolder, F.Cu at (203.8, 100.3)
- added R28: 33k, Resistor_SMD:R_0805_2012Metric_Pad1.15x1.40mm_HandSolder, B.Cu at (203.8, 113.0)
- added R29: 33k, Resistor_SMD:R_0805_2012Metric_Pad1.15x1.40mm_HandSolder, F.Cu at (203.8, 92.7)
- added R30: 33k, Resistor_SMD:R_0805_2012Metric_Pad1.15x1.40mm_HandSolder, F.Cu at (203.8, 104.1)
- added R5: 1M, Resistor_SMD:R_0805_2012Metric_Pad1.15x1.40mm_HandSolder, B.Cu at (195.8, 130.0)
- added R6: 1M, Resistor_SMD:R_0805_2012Metric_Pad1.15x1.40mm_HandSolder, B.Cu at (193.3, 130.0)
- added R7: 8k, Resistor_SMD:R_0805_2012Metric_Pad1.15x1.40mm_HandSolder, B.Cu at (205.2, 130.2)
- added R8: 33k, Resistor_SMD:R_0805_2012Metric_Pad1.15x1.40mm_HandSolder, F.Cu at (183.5, 123.8)
- added R9: 1M, Resistor_SMD:R_0805_2012Metric_Pad1.15x1.40mm_HandSolder, F.Cu at (195.8, 127.5)
- C2, C3, Q1, R1, R1a1, R2, U1, U3, U4: moved to B.Cu
- C6: footprint Capacitor_THT:C_Disc_D4.3mm_W1.9mm_P5.00mm -> Capacitor_THT:C_Disc_D6.0mm_W2.5mm_P5.00mm
- C7: footprint Capacitor_THT:C_Rect_L26.5mm_W5.0mm_P22.50mm_MKS4 -> Capacitor_THT:C_Rect_L16.5mm_W4.7mm_P15.00mm_MKT
- Q2: value MPSA42 -> MMBTA42; footprint Package_TO_SOT_THT:TO-92_Inline -> Package_TO_SOT_SMD:SOT-323_SC-70_Handsoldering; moved to B.Cu
- Q3: value MPSA92 -> MMBTA92; footprint Package_TO_SOT_THT:TO-92_Inline -> Package_TO_SOT_SMD:SOT-323_SC-70_Handsoldering; moved to B.Cu
- R3: value R -> 100k; moved to B.Cu
- R4: value 100k -> 33k; moved to B.Cu
- moved U5 168.1 mm to (145.4, 133.3), turned to 90 degrees
- moved R3 151.4 mm to (164.5, 122.3), turned to 270 degrees
- moved Q2 150.3 mm to (188.7, 130.0)
- moved T2 145.3 mm to (81.9, 59.7), turned to 90 degrees
- moved R4 143.3 mm to (184.4, 130.0), turned to 90 degrees
- moved U3 132.7 mm to (192.4, 111.1), turned to 90 degrees
- moved U1 129.7 mm to (172.3, 85.1), turned to 180 degrees
- moved Q3 123.4 mm to (200.2, 130.0)
- moved U2 123.4 mm to (190.5, 99.7), turned to 180 degrees
- moved T3 122.9 mm to (81.9, 82.5), turned to 90 degrees
- moved D5 118.9 mm to (81.9, 59.7), turned to 90 degrees
- moved T4 111.0 mm to (81.3, 119.4), turned to 90 degrees
- moved D3 109.2 mm to (81.8, 119.8), turned to 90 degrees
- moved D4 108.1 mm to (81.9, 82.5), turned to 90 degrees
- moved D2 100.4 mm to (81.7, 142.2), turned to 90 degrees
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Connections:
- net Net-(J2-Pad1) renamed /front_panel/A1
- net Net-(J2-Pad12) renamed /front_panel/D7
- net Net-(J2-Pad14) renamed /front_panel/D9
- net Net-(J2-Pad2) renamed /front_panel/A2
- net Net-(J2-Pad3) renamed /front_panel/A3
- net Net-(J2-Pad4) renamed /front_panel/A4
- net Net-(J2-Pad8) renamed /front_panel/D3
- J2 pad 10: Net-(J2-Pad10) -> /front_panel/D1
- J2 pad 11: Net-(J2-Pad11) -> /front_panel/DOT
- J2 pad 13: Net-(J2-Pad13) -> /front_panel/D0
- J2 pad 15: Net-(J2-Pad15) -> /front_panel/D6
- J2 pad 5: Net-(J2-Pad5) -> /front_panel/D4
- J2 pad 6: Net-(J2-Pad6) -> /front_panel/D5
- J2 pad 7: Net-(J2-Pad7) -> /front_panel/D8
- J2 pad 9: Net-(J2-Pad9) -> /front_panel/D2
- Q2 pad 1: GND -> Net-(Q2-Pad1)
- Q2 pad 2: Net-(Q2-Pad2) -> GND
- Q3 pad 1: /Anode1 -> Net-(Q3-Pad1)
- Q3 pad 2: Net-(Q3-Pad2) -> +VDC
- Q3 pad 3: /Vdd -> Net-(Q3-Pad3)
- R3 pad 1: Net-(Q3-Pad2) -> +3V3
- R3 pad 2: Net-(Q2-Pad3) -> Net-(R3-Pad2)
- R4 pad 1: +3V3 -> Net-(Q2-Pad1)
- R4 pad 2: Net-(R4-Pad2) -> /DRIVE_A1
- T1 pad 10: Net-(J2-Pad5) -> /front_panel/D2
- T1 pad 11: Net-(J2-Pad6) -> /front_panel/D1
- T1 pad 12: Net-(J2-Pad15) -> /front_panel/DOT
- T1 pad 2: Net-(J2-Pad7) -> /front_panel/D0
- T1 pad 4: Net-(J2-Pad13) -> /front_panel/D8
- T1 pad 6: Net-(J2-Pad11) -> /front_panel/D6
- T1 pad 7: Net-(J2-Pad10) -> /front_panel/D5
- T1 pad 8: Net-(J2-Pad9) -> /front_panel/D4
- T2 pad 10: Net-(J2-Pad5) -> /front_panel/D2
- T2 pad 11: Net-(J2-Pad6) -> /front_panel/D1
- T2 pad 12: Net-(J2-Pad15) -> /front_panel/DOT
- T2 pad 2: Net-(J2-Pad7) -> /front_panel/D0
- T2 pad 4: Net-(J2-Pad13) -> /front_panel/D8
- T2 pad 6: Net-(J2-Pad11) -> /front_panel/D6
- T2 pad 7: Net-(J2-Pad10) -> /front_panel/D5
- T2 pad 8: Net-(J2-Pad9) -> /front_panel/D4
- T3 pad 10: Net-(J2-Pad5) -> /front_panel/D2
- T3 pad 11: Net-(J2-Pad6) -> /front_panel/D1
- T3 pad 12: Net-(J2-Pad15) -> /front_panel/DOT
- T3 pad 2: Net-(J2-Pad7) -> /front_panel/D0
- T3 pad 4: Net-(J2-Pad13) -> /front_panel/D8
- T3 pad 6: Net-(J2-Pad11) -> /front_panel/D6
- T3 pad 7: Net-(J2-Pad10) -> /front_panel/D5
- T3 pad 8: Net-(J2-Pad9) -> /front_panel/D4
- T4 pad 10: Net-(J2-Pad5) -> /front_panel/D2
- T4 pad 11: Net-(J2-Pad6) -> /front_panel/D1
- T4 pad 12: Net-(J2-Pad15) -> /front_panel/DOT
- T4 pad 2: Net-(J2-Pad7) -> /front_panel/D0
- T4 pad 4: Net-(J2-Pad13) -> /front_panel/D8
- T4 pad 6: Net-(J2-Pad11) -> /front_panel/D6
- T4 pad 7: Net-(J2-Pad10) -> /front_panel/D5
- T4 pad 8: Net-(J2-Pad9) -> /front_panel/D4
- U1 pad 13: Net-(R4-Pad2) -> Net-(R3-Pad2)
- U2 pad 13: Net-(R4-Pad2) -> Net-(R3-Pad2)
- U2 pad 14: Net-(U2-Pad14) -> Net-(U1-Pad9)
- U3 pad 1: Net-(U3-Pad1) -> /DRIVE_D8
- U3 pad 13: Net-(R4-Pad2) -> Net-(R3-Pad2)
- U3 pad 14: Net-(U3-Pad14) -> Net-(U2-Pad9)
- U3 pad 15: Net-(U3-Pad15) -> /DRIVE_D3
- U3 pad 2: Net-(U3-Pad2) -> /DRIVE_D5
- U3 pad 3: Net-(U3-Pad3) -> /DRIVE_D4
- U3 pad 4: Net-(U3-Pad4) -> /DRIVE_A4
- U3 pad 5: Net-(U3-Pad5) -> /DRIVE_A3
- U3 pad 6: Net-(U3-Pad6) -> /DRIVE_A2
- U3 pad 7: Net-(U3-Pad7) -> /DRIVE_A1
- U5 pad 3: /+9V -> +9V
Routing:
- net Net-(J2-Pad15): track 230.7 -> 0.00 mm, vias 6 -> 0
- net /front_panel/D6: track 0.00 -> 230.7 mm, vias 0 -> 6
- net Net-(J2-Pad7): track 198.9 -> 0.00 mm, vias 5 -> 0
- net /front_panel/D8: track 0.00 -> 198.9 mm, vias 0 -> 5
- net Net-(J2-Pad6): track 191.3 -> 0.00 mm, vias 5 -> 0
- net /front_panel/D5: track 0.00 -> 191.3 mm, vias 0 -> 5
- net Net-(J2-Pad5): track 189.5 -> 0.00 mm, vias 5 -> 0
- net /front_panel/D4: track 0.00 -> 189.5 mm, vias 0 -> 5
- net Net-(J2-Pad9): track 158.0 -> 0.00 mm, vias 6 -> 0
- net /front_panel/D2: track 0.00 -> 158.0 mm, vias 0 -> 6
- net Net-(J2-Pad10): track 153.7 -> 0.00 mm, vias 6 -> 0
- net /front_panel/D1: track 0.00 -> 153.7 mm, vias 0 -> 6
- net Net-(J2-Pad11): track 152.2 -> 0.00 mm, vias 4 -> 0
- net /front_panel/DOT: track 0.00 -> 152.2 mm, vias 0 -> 4
- net Net-(J2-Pad13): track 151.5 -> 0.00 mm, vias 6 -> 0
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- added copper zone on B.Cu, net GND
- added copper zone on F.Cu, net GND
Other:
- board size 80 x 130 mm -> 170.8 x 131.9 mm
- net class Default: clearance 0.6 -> 0.4; trace_width 0.6 -> 0.4
- rule trace_clearance: 0.6 -> 0.4

Commit message: Schematic complete. PCB nearly done.
Parts:
- added C1: 100n, Capacitor_SMD:C_1206_3216Metric_Pad1.42x1.75mm_HandSolder, F.Cu at (169.7, 70.1)
- added C10: 100n, Capacitor_SMD:C_1206_3216Metric_Pad1.42x1.75mm_HandSolder, B.Cu at (172.7, 94.5)
- added C8: 100n, Capacitor_SMD:C_1206_3216Metric_Pad1.42x1.75mm_HandSolder, B.Cu at (168.7, 75.7)
- added C9: 100n, Capacitor_SMD:C_1206_3216Metric_Pad1.42x1.75mm_HandSolder, B.Cu at (172.8, 113.8)
- added D6: 1N4763A 91V, Diode_SMD:D_MiniMELF_Handsoldering, B.Cu at (203.0, 92.1)
- added D7: 1N4763A 91V, Diode_SMD:D_MiniMELF_Handsoldering, B.Cu at (203.2, 87.0)
- added FLASH1: SW_DIP_x01, Button_Switch_THT:SW_PUSH_6mm, F.Cu at (156.0, 36.6)
- added J4: Conn_01x04_Male, Connector_PinHeader_2.54mm:PinHeader_1x05_P2.54mm_Horizontal, F.Cu at (166.6, 44.2)
- added Q21: MMBTA42, Package_TO_SOT_SMD:SOT-323_SC-70_Handsoldering, B.Cu at (194.9, 92.1)
- added Q22: MMBTA42, Package_TO_SOT_SMD:SOT-323_SC-70_Handsoldering, B.Cu at (195.0, 87.0)
- added R31: 10k, Resistor_SMD:R_0805_2012Metric_Pad1.15x1.40mm_HandSolder, B.Cu at (188.0, 45.2)
- added R32: 10k, Resistor_SMD:R_0805_2012Metric_Pad1.15x1.40mm_HandSolder, B.Cu at (160.0, 44.7)
- added R33: 0R0, Resistor_SMD:R_0805_2012Metric_Pad1.15x1.40mm_HandSolder, B.Cu at (154.4, 83.3)
- added R34: 0R0, Resistor_SMD:R_0805_2012Metric_Pad1.15x1.40mm_HandSolder, B.Cu at (153.4, 87.4)
- added R35: 10k, Resistor_SMD:R_0805_2012Metric_Pad1.15x1.40mm_HandSolder, F.Cu at (155.4, 75.2)
- added R36: 4k7, Resistor_SMD:R_0805_2012Metric_Pad1.15x1.40mm_HandSolder, F.Cu at (147.8, 78.2)
- added R37: 12k, Resistor_SMD:R_0805_2012Metric_Pad1.15x1.40mm_HandSolder, F.Cu at (150.9, 77.2)
- added R38: R_PHOTO, OptoDevice:R_LDR_4.9x4.2mm_P2.54mm_Vertical, F.Cu at (144.3, 77.2)
- added R39: 10k, Resistor_SMD:R_0805_2012Metric_Pad1.15x1.40mm_HandSolder, B.Cu at (167.6, 51.3)
- added R40: 33k, Resistor_SMD:R_0805_2012Metric_Pad1.15x1.40mm_HandSolder, B.Cu at (189.9, 92.7)
- added R41: 33k, Resistor_SMD:R_0805_2012Metric_Pad1.15x1.40mm_HandSolder, B.Cu at (189.9, 87.6)
- added R42: 240k, Resistor_SMD:R_0805_2012Metric_Pad1.15x1.40mm_HandSolder, F.Cu at (210.8, 88.3)
- added R43: 240k, Resistor_SMD:R_0805_2012Metric_Pad1.15x1.40mm_HandSolder, F.Cu at (210.8, 83.2)
- added R44: 68R, Resistor_SMD:R_0805_2012Metric_Pad1.15x1.40mm_HandSolder, B.Cu at (208.3, 81.9)
- added R45: 15R, Resistor_SMD:R_0805_2012Metric_Pad1.15x1.40mm_HandSolder, B.Cu at (208.3, 79.4)
- added R46: 15R, Resistor_SMD:R_0805_2012Metric_Pad1.15x1.40mm_HandSolder, B.Cu at (208.3, 76.8)
- added RST1: SW_DIP_x01, Button_Switch_THT:SW_PUSH_6mm, F.Cu at (180.8, 36.6)
- added U6: ESP-12E, ESP8266:ESP-12E_SMD, F.Cu at (150.0, 70.0)
- Q10, Q11, Q12, Q17, Q19, Q20, R20, R21, R22, R27, R29, R30, U2: moved to B.Cu
- R3: value 100k -> 10k
- moved J1 124.4 mm to (201.7, 38.1), turned to 270 degrees
- moved U5 86.3 mm to (186.5, 57.4), turned to 180 degrees
- moved R2 53.5 mm to (131.4, 180.3)
- moved RSENSE1 53.5 mm to (151.8, 188.0)
- moved U4 53.5 mm to (144.1, 182.2)
- moved C2 53.5 mm to (135.9, 183.5)
- moved C4 53.5 mm to (129.5, 187.3)
- moved C6 53.5 mm to (133.3, 171.4)
- moved L1 53.5 mm to (129.5, 193.0)
- moved Q1 53.5 mm to (144.1, 194.1)
- moved R1a1 53.5 mm to (136.3, 180.3)
- moved C5 53.5 mm to (158.1, 176.5)
- moved C7 53.5 mm to (158.1, 188.6)
- moved D1 53.5 mm to (153.0, 198.5)
- moved R1 53.5 mm to (137.2, 175.3)
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Connections:
- net +VDC renamed 180V
- J3 pad 16: Net-(J3-Pad16) -> /ANODE_N1
- J3 pad 17: Net-(J3-Pad17) -> /CATHODE_N1
- J3 pad 18: Net-(J3-Pad18) -> /ANODE_N2
- J3 pad 19: Net-(J3-Pad19) -> /CATHODE_N2
- J3 pad 20: Net-(J3-Pad20) -> /RED
- J3 pad 21: Net-(J3-Pad21) -> /GREEN
- J3 pad 22: Net-(J3-Pad22) -> /BLUE
- J3 pad 23: Net-(J3-Pad23) -> /DRIVE_LED_A1
- J3 pad 24: Net-(J3-Pad24) -> /DRIVE_LED_A2
- J3 pad 25: Net-(J3-Pad25) -> /DRIVE_LED_A3
- J3 pad 26: Net-(J3-Pad26) -> /DRIVE_LED_A4
- R3 pad 2: Net-(R3-Pad2) -> BLANK
- U1 pad 1: Net-(U1-Pad1) -> /DRIVE_LED_A3
- U1 pad 10: Net-(U1-Pad10) -> GND
- U1 pad 11: Net-(U1-Pad11) -> HSPI_CLK
- U1 pad 12: Net-(U1-Pad12) -> HSPI_CS
- U1 pad 13: Net-(R3-Pad2) -> Net-(R33-Pad1)
- U1 pad 14: Net-(U1-Pad14) -> HSPI_MOSI
- U1 pad 15: Net-(U1-Pad15) -> /DRIVE_LED_A4
- U1 pad 2: Net-(U1-Pad2) -> /DRIVE_LED_A2
- U1 pad 3: Net-(U1-Pad3) -> /DRIVE_LED_A1
- U1 pad 4: Net-(U1-Pad4) -> /DRIVE_BLUE
- U1 pad 5: Net-(U1-Pad5) -> /DRIVE_GREEN
- U1 pad 6: Net-(U1-Pad6) -> /DRIVE_RED
- U1 pad 7: Net-(U1-Pad7) -> /DRIVE_S2
- U2 pad 1: Net-(U2-Pad1) -> /DRIVE_D6
- U2 pad 10: Net-(U2-Pad10) -> GND
- U2 pad 11: Net-(U2-Pad11) -> HSPI_CLK
- U2 pad 12: Net-(U2-Pad12) -> HSPI_CS
- U2 pad 13: Net-(R3-Pad2) -> Net-(R33-Pad1)
- U2 pad 15: Net-(U2-Pad15) -> /DRIVE_S1
- U2 pad 2: Net-(U2-Pad2) -> /DRIVE_D9
- U2 pad 3: Net-(U2-Pad3) -> /DRIVE_D0
- U2 pad 4: Net-(U2-Pad4) -> /DRIVE_D7
- U2 pad 5: Net-(U2-Pad5) -> /DRIVE_DOT
- U2 pad 6: Net-(U2-Pad6) -> /DRIVE_D1
- U2 pad 7: Net-(U2-Pad7) -> /DRIVE_D2
- U3 pad 10: Net-(U3-Pad10) -> GND
- U3 pad 11: Net-(U3-Pad11) -> HSPI_CLK
- U3 pad 12: Net-(U3-Pad12) -> HSPI_CS
- U3 pad 13: Net-(R3-Pad2) -> Net-(R33-Pad1)
- U4 pad 4: GND -> Net-(R34-Pad1)
Routing:
- net +3V3: track 15.4 -> 169.9 mm, vias 0 -> 5
- net HSPI_CS: track 0.00 -> 97.2 mm, vias 0 -> 5
- net RESET: track 0.00 -> 84.0 mm, vias 0 -> 1
- net HSPI_CLK: track 0.00 -> 78.2 mm, vias 0 -> 4
- net Net-(R33-Pad1): track 0.00 -> 66.5 mm, vias 0 -> 3
- net /DRIVE_LED_A4: track 0.00 -> 50.7 mm
- net /DRIVE_LED_A3: track 0.00 -> 43.1 mm
- net BLANK: track 0.00 -> 42.6 mm, vias 0 -> 1
- net /DRIVE_LED_A2: track 0.00 -> 42.6 mm
- net /DRIVE_LED_A1: track 0.00 -> 42.0 mm
- net 180V: track 131.3 -> 172.7 mm
- net +9V: track 19.4 -> 52.5 mm
- net /DRIVE_BLUE: track 0.00 -> 33.0 mm
- net /DRIVE_GREEN: track 0.00 -> 32.5 mm
- net Net-(J4-Pad3): track 0.00 -> 32.5 mm, vias 0 -> 1
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Other:
- net class Default: clearance 0.4 -> 0.3
- rule trace_clearance: 0.4 -> 0.3
- board text added: "+3V3"
- board text added: "180V"
- board text added: "GND"
- board text added: "N/A"
- board text added: "RX"
- board text added: "TX"
- board text added: "flash"
- board text added: "reset"

Commit message: First final draft ready (Ausf B)
Parts:
- added C11: 10uF, Capacitor_THT:CP_Radial_D5.0mm_P2.50mm, F.Cu at (194.6, 55.9)
- added C12: 22uF, Capacitor_THT:CP_Radial_D5.0mm_P2.50mm, F.Cu at (185.5, 64.0)
- added C13: 10uF,25V, Capacitor_THT:CP_Radial_D5.0mm_P2.50mm, F.Cu at (174.8, 132.6)
- added U7: THERMAL_VIA, PartsStash_RW:Thermal_Via, F.Cu at (192.0, 62.0)
- C8: moved to F.Cu
- L1: footprint Inductor_THT:L_Toroid_Vertical_L16.0mm_W8.0mm_P7.62mm -> PartsStash_RW:L_Toroid_Horizontal_D16.8mm_P6mm_AliExpress
- RSENSE1: footprint Resistor_THT:R_Axial_DIN0516_L15.5mm_D5.0mm_P5.08mm_Vertical -> Resistor_THT:R_Axial_DIN0414_L11.9mm_D4.5mm_P15.24mm_Horizontal
- moved C7 61.8 mm to (201.7, 144.8)
- moved C5 55.8 mm to (198.6, 138.2)
- moved D1 55.6 mm to (191.6, 158.5), turned to 180 degrees
- moved C3 55.5 mm to (181.9, 135.6), turned to 0 degrees
- moved L1 55.2 mm to (159.0, 146.3), turned to 270 degrees
- moved U4 53.5 mm to (177.6, 140.6)
- moved Q1 53.5 mm to (177.7, 152.5)
- moved C2 51.4 mm to (169.7, 144.7), turned to 270 degrees
- moved C4 50.4 mm to (152.9, 142.7)
- moved RSENSE1 50.0 mm to (188.0, 153.4)
- moved R1 49.2 mm to (164.1, 134.1)
- moved R1a1 49.1 mm to (163.1, 139.2)
- moved R2 49.0 mm to (158.0, 139.2)
- moved C6 48.8 mm to (160.0, 130.6)
- moved C8 4.60 mm to (168.1, 80.3), turned to 270 degrees
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Routing:
- net +9V: track 52.5 -> 168.8 mm, vias 0 -> 2
- net Net-(R34-Pad1): track 5.98 -> 62.2 mm
- net 180V: track 172.7 -> 200.5 mm, vias 2 -> 4
- net +3V3: track 169.9 -> 179.1 mm, vias 5 -> 6
- net Net-(Q1-Pad3): track 9.47 -> 18.3 mm
- net Net-(C6-Pad2): track 11.5 -> 18.8 mm
- net Net-(D1-Pad2): track 27.2 -> 31.4 mm
- net Net-(Q4-Pad1): track 0.00 -> 3.06 mm
- net Net-(R1a1-Pad2): track 0.00 -> 3.03 mm
- net /CATHODE_N2: track 21.2 -> 22.0 mm
- net GND: vias 1 -> 0
