File: kicad/funknetzwerkuhr.kicad_pcb (KiCad board)
At the start: 2 copper layers, 170.8 x 131.9 mm, 110 parts, among them J1 Jack-DC, J2 Conn_01x26_Male, J3 Conn_01x26_Female, J4 Conn_01x04_Male, Q1 IRF640, Q10 MMBTA42, Q11 MMBTA42, Q12 MMBTA42, Q13 MMBTA42, Q14 MMBTA42, Q15 MMBTA42, Q16 MMBTA42, Q17 MMBTA42, Q18 MMBTA42, Q19 MMBTA42, Q2 MMBTA42, Q20 MMBTA42, Q21 MMBTA42, Q22 MMBTA42, Q3 MMBTA92, Q4 MMBTA42, Q5 MMBTA92, Q6 MMBTA42, Q7 MMBTA92, Q8 MMBTA42, Q9 MMBTA92, T1 IN-12, T2 IN-12, T3 IN-12, T4 IN-12, U1 74HC595, U2 74HC595, U3 74HC595, U4 max1771, U5 AP1117-33, U6 ESP-12E, U7 THERMAL_VIA

Commit message: Nothing works now.
Parts:
- added U10: THERMAL_VIA, PartsStash_RW:Thermal_Via, F.Cu at (180.3, 74.3)
- added U11: THERMAL_VIA, PartsStash_RW:Thermal_Via, F.Cu at (175.9, 110.7)
- added U12: THERMAL_VIA, PartsStash_RW:Thermal_Via, F.Cu at (179.7, 67.3)
- added U13: THERMAL_VIA, PartsStash_RW:Thermal_Via, F.Cu at (196.2, 49.5)
- added U14: THERMAL_VIA, PartsStash_RW:Thermal_Via, F.Cu at (202.2, 134.6)
- added U15: THERMAL_VIA, PartsStash_RW:Thermal_Via, F.Cu at (212.1, 128.9)
- added U16: THERMAL_VIA, PartsStash_RW:Thermal_Via, F.Cu at (212.1, 123.2)
- added U8: THERMAL_VIA, PartsStash_RW:Thermal_Via, F.Cu at (175.9, 90.8)
- added U9: THERMAL_VIA, PartsStash_RW:Thermal_Via, F.Cu at (175.3, 128.3)
- C8: moved to B.Cu
- FLASH1, RST1: footprint Button_Switch_THT:SW_PUSH_6mm -> Button_Switch_THT:SW_PUSH-12mm
- Q10, Q11, Q12, Q13, Q14, Q15, Q16, Q17, Q18, Q19, Q2, Q20, Q21, Q22, Q3, Q4, Q5, Q6, Q7, Q8, Q9: footprint Package_TO_SOT_SMD:SOT-323_SC-70_Handsoldering -> Package_TO_SOT_SMD:TSOT-23_HandSoldering
- U5: value AP1117-33 -> NCP1117-33G; footprint Package_TO_SOT_SMD:SOT-223-3_TabPin2 -> PartsStash_RW:DPACK2
- moved U7 22.5 mm to (170.2, 67.3)
- moved C8 8.97 mm to (174.8, 74.3), turned to 0 degrees
- moved FLASH1 5.34 mm to (150.7, 37.5)
- moved J1 3.64 mm to (205.3, 38.1)
- moved R32 3.24 mm to (162.3, 47.0)
- moved U5 2.90 mm to (184.2, 59.1), turned to 90 degrees
- moved R39 2.79 mm to (165.7, 53.3)
- moved C5 2.23 mm to (196.8, 136.8), turned to 270 degrees
- moved RST1 1.83 mm to (182.4, 37.5)
- moved C11 1.75 mm to (196.2, 56.5), turned to 180 degrees
- moved C4 1.72 mm to (152.9, 141.0), turned to 180 degrees
- moved C12 1.55 mm to (184.8, 65.4)
- moved C9 1.45 mm to (174.2, 113.8)
- moved R37 1.43 mm to (151.8, 78.3)
- moved R36 1.40 mm to (149.2, 78.2)
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Routing:
- net 180V: track 200.5 -> 179.3 mm, vias 4 -> 1
- net +3V3: track 179.1 -> 165.3 mm, vias 6 -> 4
- net RESET: track 84.0 -> 94.6 mm
- net +9V: track 168.8 -> 175.1 mm
- net HSPI_CS: track 97.2 -> 92.0 mm
- net BLANK: track 42.6 -> 39.1 mm
- net FLASH: track 27.3 -> 30.0 mm
- net ADC: track 13.7 -> 16.2 mm
- net Net-(C6-Pad2): track 18.8 -> 20.1 mm
- net Net-(J4-Pad3): track 32.5 -> 31.8 mm
- net /DRIVE_D8: track 28.6 -> 29.2 mm
- net /DRIVE_LED_A4: track 50.7 -> 50.1 mm
- net HSPI_MOSI: track 22.1 -> 22.7 mm
- net /DRIVE_D6: track 29.6 -> 30.1 mm
- net /DRIVE_D0: track 28.6 -> 29.1 mm
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- added copper zone on F.Cu, net +3V3
- added copper zone on F.Cu, net +9V
- added copper zone on F.Cu, net 180V
Other:
- board text added: "DC IN"
