File: kicad/hv_psu.sch (KiCad schematic (older format))
At the start: 16 parts, among them J1 Jack-DC, Q1 IRF640, U4 max1771

Commit message: Schematic nearly done, need to add programming header.
Parts:
- removed C1: 10uF,25V, Capacitor_THT:CP_Radial_D5.0mm_P2.50mm, symbol Device:CP
- added R34: 0R0, Resistor_SMD:R_0805_2012Metric_Pad1.15x1.40mm_HandSolder, symbol Device:R
- C6: footprint (none) -> Capacitor_THT:C_Disc_D6.0mm_W2.5mm_P5.00mm
- C7: footprint Capacitor_THT:C_Rect_L26.5mm_W5.0mm_P22.50mm_MKS4 -> Capacitor_THT:C_Rect_L16.5mm_W4.7mm_P15.00mm_MKT
- R1a1, R2: footprint Resistor_SMD:R_0805_2012Metric_Pad1.33x1.40mm_HandSolder -> Resistor_SMD:R_0805_2012Metric_Pad1.15x1.40mm_HandSolder
Connections:
- net labels added: BLANK
- wire segments 67 -> 62
Changed lines of the file:
@@
 EESchema Schematic File Version 4
 LIBS:funknetzwerkuhr-cache
-LIBS:nixie-breakout-cache
 EELAYER 26 0
 EELAYER END
 $Descr A4 11693 8268
 encoding utf-8
-Sheet 2 4
+Sheet 2 3
 Title ""
 Date ""
@@
 	1    0    0    -1
 $EndComp
-Wire Wire Line
-	5100 3600 4400 3600
 $Comp
 L Device:C C3
@@
 Connection ~ 5550 2700
 Wire Wire Line
-	4400 4550 4050 4550
+	4400 4550 3900 4550
 $Comp
 L Device:C C2
 U 1 1 5B78B212
-P 4050 3450
-F 0 "C2" V 4150 3300 50  0000 L CNN
-F 1 "100n" V 3900 3350 50  0000 L CNN
-F 2 "Capacitor_SMD:C_1206_3216Metric_Pad1.42x1.75mm_HandSolder" H 4088 3300 50  0001 C CNN
-F 3 "" H 4050 3450 50  0001 C CNN
-	1    4050 3450
-	1    0    0    -1
-$EndComp
-$Comp
-L Device:CP C1
-U 1 1 5B78B6C2
-P 3650 3450
-F 0 "C1" V 3750 3300 50  0000 L CNN
-F 1 "10uF,25V" V 3500 3300 50  0000 L CNN
-F 2 "Capacitor_THT:CP_Radial_D5.0mm_P2.50mm" H 3688 3300 50  0001 C CNN
-F 3 "" H 3650 3450 50  0001 C CNN
-	1    3650 3450
-	1    0    0    -1
-$EndComp
-Wire Wire Line
-	3650 3300 3650 2700
-Wire Wire Line
-	3650 2700 4050 2700
-Wire Wire Line
-	4050 3300 4050 2700
-Connection ~ 4050 2700
-Wire Wire Line
-	4050 2700 5550 2700
-Wire Wire Line
-	4050 3600 4050 4550
-Connection ~ 4050 4550
-Wire Wire Line
-	4050 4550 3650 4550
-Wire Wire Line
-	3650 3600 3650 4550
+P 3500 3500
+F 0 "C2" V 3600 3350 50  0000 L CNN
+F 1 "100n" V 3350 3400 50  0000 L CNN
+F 2 "Capacitor_SMD:C_1206_3216Metric_Pad1.42x1.75mm_HandSolder" H 3538 3350 50  0001 C CNN
+F 3 "" H 3500 3500 50  0001 C CNN
+	1    3500 3500
+	1    0    0    -1
+$EndComp
+Wire Wire Line
+	3500 3350 3500 2700
+Wire Wire Line
+	3500 2700 3900 2700
+Wire Wire Line
+	3500 3650 3500 4550
 $Comp
 L Device:L L1
@@
 L Device:CP C4
 U 1 1 5B7B059A
-P 5900 2950
-F 0 "C4" V 6000 2800 50  0000 L CNN
-F 1 "100uF,25V" V 5750 2800 50  0000 L CNN
-F 2 "Capacitor_THT:CP_Radial_D8.0mm_P3.50mm" H 5938 2800 50  0001 C CNN
-F 3 "" H 5900 2950 50  0001 C CNN
-	1    5900 2950
-	1    0    0    -1
-$EndComp
-$Comp
-L power:GND #PWR012
-U 1 1 5B7B0698
-P 5900 3150
-F 0 "#PWR012" H 5900 2900 50  0001 C CNN
-F 1 "GND" H 5905 2977 50  0000 C CNN
-F 2 "" H 5900 3150 50  0001 C CNN
-F 3 "" H 5900 3150 50  0001 C CNN
-	1    5900 3150
-	1    0    0    -1
-$EndComp
-Wire Wire Line
-	6100 2700 5900 2700
+P 3900 3500
+F 0 "C4" V 4000 3350 50  0000 L CNN
+F 1 "100uF,25V" V 3750 3350 50  0000 L CNN
+F 2 "Capacitor_THT:CP_Radial_D8.0mm_P3.50mm" H 3938 3350 50  0001 C CNN
+F 3 "" H 3900 3500 50  0001 C CNN
+	1    3900 3500
+	1    0    0    -1
+$EndComp
 Wire Wire Line
 	5550 2550 5550 2700
-Wire Wire Line
-	5900 2800 5900 2700
-Connection ~ 5900 2700
-Wire Wire Line
-	5900 2700 5550 2700
-Wire Wire Line
-	5900 3150 5900 3100
 $Comp
 L Transistor_FET:IRF740 Q1
@@
 F 0 "R2" H 7770 4346 50  0000 L CNN
 F 1 "10k" H 7770 4255 50  0000 L CNN
-F 2 "Resistor_SMD:R_0805_2012Metric_Pad1.33x1.40mm_HandSolder" V 7630 4300 50  0001 C CNN
+F 2 "Resistor_SMD:R_0805_2012Metric_Pad1.15x1.40mm_HandSolder" V 7630 4300 50  0001 C CNN
 F 3 "" H 7700 4300 50  0001 C CNN
 	1    7700 4300
@@
 	7700 2700 7300 2700
 Connection ~ 7300 2700
-Wire Wire Line
-	4400 3600 4400 4550
 Wire Wire Line
 	6000 4050 6950 4050
@@
 F 0 "C7" V 8650 3450 50  0000 L CNN
 F 1 "100n,250V" V 8400 3400 50  0000 L CNN
-F 2 "Capacitor_THT:C_Rect_L26.5mm_W5.0mm_P22.50mm_MKS4" H 8588 3450 50  0001 C CNN
+F 2 "Capacitor_THT:C_Rect_L16.5mm_W4.7mm_P15.00mm_MKT" H 8588 3450 50  0001 C CNN
 F 3 "" H 8550 3600 50  0001 C CNN
 	1    8550 3600
@@
 F 0 "R1a1" H 7770 3946 50  0000 L CNN
 F 1 "2.7k" H 7770 3855 50  0000 L CNN
-F 2 "Resistor_SMD:R_0805_2012Metric_Pad1.33x1.40mm_HandSolder" V 7630 3900 50  0001 C CNN
+F 2 "Resistor_SMD:R_0805_2012Metric_Pad1.15x1.40mm_HandSolder" V 7630 3900 50  0001 C CNN
 F 3 "" H 7700 3900 50  0001 C CNN
 	1    7700 3900
@@
 F 0 "C6" H 8165 3146 50  0000 L CNN
 F 1 "100p 1kV" H 8165 3055 50  0000 L CNN
-F 2 "" H 8088 2950 50  0001 C CNN
+F 2 "Capacitor_THT:C_Disc_D6.0mm_W2.5mm_P5.00mm" H 8088 2950 50  0001 C CNN
 F 3 "~" H 8050 3100 50  0001 C CNN
 	1    8050 3100
@@
 	4200 2050 4100 2050
 Connection ~ 4100 2050
+Wire Wire Line
+	3900 3650 3900 4550
+Connection ~ 3900 4550
+Wire Wire Line
+	3900 4550 3500 4550
+Wire Wire Line
+	5550 2700 6100 2700
+Wire Wire Line
+	3900 3350 3900 2700
+Connection ~ 3900 2700
+Wire Wire Line
+	3900 2700 5550 2700
+Text GLabel 4800 3600 0    50   Input ~ 0
+BLANK
+$Comp
+L Device:R R34
+U 1 1 5B6FD7F5
+P 4950 3600
+F 0 "R34" V 4743 3600 50  0000 C CNN
+F 1 "0R0" V 4834 3600 50  0000 C CNN
+F 2 "Resistor_SMD:R_0805_2012Metric_Pad1.15x1.40mm_HandSolder" V 4880 3600 50  0001 C CNN
+F 3 "~" H 4950 3600 50  0001 C CNN
+	1    4950 3600
+	0    1    1    0
+$EndComp
 $EndSCHEMATC

Commit message: First final draft ready (Ausf B)
Parts:
- added C13: 10uF,25V, Capacitor_THT:CP_Radial_D5.0mm_P2.50mm, symbol Device:CP
- L1: footprint Inductor_THT:L_Toroid_Vertical_L16.0mm_W8.0mm_P7.62mm -> PartsStash_RW:L_Toroid_Horizontal_D16.8mm_P6mm_AliExpress
- RSENSE1: footprint Resistor_THT:R_Axial_DIN0516_L15.5mm_D5.0mm_P5.08mm_Vertical -> Resistor_THT:R_Axial_DIN0414_L11.9mm_D4.5mm_P15.24mm_Horizontal
Connections:
- wire segments 62 -> 63
Changed lines of the file:
@@
 $Descr A4 11693 8268
 encoding utf-8
-Sheet 2 3
+Sheet 3 3
 Title ""
 Date ""
@@
 F 0 "L1" V 6440 2700 50  0000 C CNN
 F 1 "L" V 6349 2700 50  0000 C CNN
-F 2 "Inductor_THT:L_Toroid_Vertical_L16.0mm_W8.0mm_P7.62mm" H 6250 2700 50  0001 C CNN
+F 2 "PartsStash_RW:L_Toroid_Horizontal_D16.8mm_P6mm_AliExpress" H 6250 2700 50  0001 C CNN
 F 3 "" H 6250 2700 50  0001 C CNN
 	1    6250 2700
@@
 L Device:CP C4
 U 1 1 5B7B059A
-P 3900 3500
-F 0 "C4" V 4000 3350 50  0000 L CNN
-F 1 "100uF,25V" V 3750 3350 50  0000 L CNN
-F 2 "Capacitor_THT:CP_Radial_D8.0mm_P3.50mm" H 3938 3350 50  0001 C CNN
-F 3 "" H 3900 3500 50  0001 C CNN
-	1    3900 3500
+P 5900 2850
+F 0 "C4" V 6000 2700 50  0000 L CNN
+F 1 "100uF,25V" V 5750 2700 50  0000 L CNN
+F 2 "Capacitor_THT:CP_Radial_D8.0mm_P3.50mm" H 5938 2700 50  0001 C CNN
+F 3 "" H 5900 2850 50  0001 C CNN
+	1    5900 2850
 	1    0    0    -1
 $EndComp
@@
 F 0 "RSENSE1" V 6500 4200 50  0000 L CNN
 F 1 "0R1" V 6700 4200 50  0000 L CNN
-F 2 "Resistor_THT:R_Axial_DIN0516_L15.5mm_D5.0mm_P5.08mm_Vertical" V 6530 4300 50  0001 C CNN
+F 2 "Resistor_THT:R_Axial_DIN0414_L11.9mm_D4.5mm_P15.24mm_Horizontal" V 6530 4300 50  0001 C CNN
 F 3 "" H 6600 4300 50  0001 C CNN
 	1    6600 4300
@@
 	3900 4550 3500 4550
 Wire Wire Line
-	5550 2700 6100 2700
+	5550 2700 5900 2700
 Wire Wire Line
 	3900 3350 3900 2700
@@
 	0    1    1    0
 $EndComp
+Connection ~ 5900 2700
+Wire Wire Line
+	5900 2700 6100 2700
+$Comp
+L power:GND #PWR049
+U 1 1 5B7288C4
+P 5900 3000
+F 0 "#PWR049" H 5900 2750 50  0001 C CNN
+F 1 "GND" H 5905 2827 50  0000 C CNN
+F 2 "" H 5900 3000 50  0001 C CNN
+F 3 "" H 5900 3000 50  0001 C CNN
+	1    5900 3000
+	1    0    0    -1
+$EndComp
+$Comp
+L Device:CP C13
+U 1 1 5B7288EF
+P 3900 3500
+F 0 "C13" V 4000 3350 50  0000 L CNN
+F 1 "10uF,25V" V 3750 3350 50  0000 L CNN
+F 2 "Capacitor_THT:CP_Radial_D5.0mm_P2.50mm" H 3938 3350 50  0001 C CNN
+F 3 "" H 3900 3500 50  0001 C CNN
+	1    3900 3500
+	1    0    0    -1
+$EndComp
 $EndSCHEMATC
