File: kicad/funknetzwerkuhr.sch (KiCad schematic (older format))
At the start: 8 parts, among them U1 74HC595, U2 74HC595, U3 74HC595, U5 AP1117-33

Commit message: Schematic nearly done, need to add programming header.
Parts:
- added Q10, Q11, Q12, Q13, Q14, Q15, Q16, Q17, Q18, Q19, Q20, Q4, Q6, Q8: MMBTA42, Package_TO_SOT_SMD:SOT-323_SC-70_Handsoldering, symbol Parts_Stash:MMBTA42
- added Q5, Q7, Q9: MMBTA92, Package_TO_SOT_SMD:SOT-323_SC-70_Handsoldering, symbol Parts_Stash:MMBTA92
- added R10, R13, R14, R17, R18, R5, R9: 1M, Resistor_SMD:R_0805_2012Metric_Pad1.15x1.40mm_HandSolder, symbol Device:R
- added R11, R15, R19, R7: 8k, Resistor_SMD:R_0805_2012Metric_Pad1.15x1.40mm_HandSolder, symbol Device:R
- added R12, R16, R20, R21, R22, R23, R24, R25, R26, R27, R28, R29, R30, R4, R8: 33k, Resistor_SMD:R_0805_2012Metric_Pad1.15x1.40mm_HandSolder, symbol Device:R
- added R31, R32, R35: 10k, Resistor_SMD:R_0805_2012Metric_Pad1.15x1.40mm_HandSolder, symbol Device:R
- added R33: 0R0, Resistor_SMD:R_0805_2012Metric_Pad1.15x1.40mm_HandSolder, symbol Device:R
- added R36: 4k7, Resistor_SMD:R_0805_2012Metric_Pad1.15x1.40mm_HandSolder, symbol Device:R
- added R37: 12k, Resistor_SMD:R_0805_2012Metric_Pad1.15x1.40mm_HandSolder, symbol Device:R
- added R38: R_PHOTO, symbol Device:R_PHOTO
- added SW1: SW_DIP_x01, symbol Switch:SW_DIP_x01
- added SW2: SW_DIP_x01, Button_Switch_THT:SW_PUSH_6mm, symbol Switch:SW_DIP_x01
- added U6: ESP-12E, ESP8266:ESP-12E_SMD, symbol ESP8266:ESP-12E
- Q2: renamed from Q?; value MPSA42 -> MMBTA42; footprint Package_TO_SOT_THT:TO-92_Inline -> Package_TO_SOT_SMD:SOT-323_SC-70_Handsoldering; symbol Transistor_BJT:MPSA42 -> Parts_Stash:MMBTA42
- Q3: renamed from Q?; value MPSA92 -> MMBTA92; footprint Package_TO_SOT_THT:TO-92_Inline -> Package_TO_SOT_SMD:SOT-323_SC-70_Handsoldering; symbol Transistor_BJT:MPSA92 -> Parts_Stash:MMBTA92
- R3: renamed from R?; value 100k -> 10k
- R6: renamed from R?; value R -> 1M
- renumbered U3 to U1, U1 to U3
Connections:
- net labels added: 180V, 9V, A1, A2, A3, A4, ADC, BLANK, D0, D1, D2, D3, D4, D5, D6, D7, D8, D9, DOT, DRIVE_A1, DRIVE_A2, DRIVE_A3, DRIVE_A4, DRIVE_D0, DRIVE_D1, DRIVE_D2, DRIVE_D3, DRIVE_D4, DRIVE_D5, DRIVE_D6, DRIVE_D7, DRIVE_D8, DRIVE_D9, DRIVE_DOT, FLASH, HSPI_CLK, HSPI_CS, HSPI_MOSI, RESET
- net labels removed: +9V, Anode1, Vdd
- wire segments 28 -> 173
Other:
- moved on the sheet: U5

Commit message: Added 1st prototype of clock's brains.
Parts:
- added J?: Conn_01x04_Male, symbol Connector:Conn_01x04_Male
- added R39: 10k, Resistor_SMD:R_0805_2012Metric_Pad1.15x1.40mm_HandSolder, symbol Device:R
Connections:
- wire segments 173 -> 179
Changed lines of the file:
@@
 Text GLabel 1500 1850 0    50   Input ~ 0
 HSPI_MOSI
-Text GLabel 3300 1850 2    50   Input ~ 0
+Text GLabel 3600 1850 2    50   Input ~ 0
 HSPI_CS
 Text GLabel 9350 3000 1    50   Input ~ 0
@@
 Wire Wire Line
 	1500 1950 950  1950
-Wire Bus Line
-	1650 6400 10900 6400
-Wire Bus Line
-	9700 800  9700 2650
-Wire Bus Line
-	1600 4500 10350 4500
 $Comp
 L power:+3V3 #PWR036
@@
 	1    0    0    -1
 $EndComp
+$Comp
+L Device:R R39
+U 1 1 5B63E588
+P 3450 2000
+F 0 "R39" H 3520 2046 50  0000 L CNN
+F 1 "10k" H 3520 1955 50  0000 L CNN
+F 2 "Resistor_SMD:R_0805_2012Metric_Pad1.15x1.40mm_HandSolder" V 3380 2000 50  0001 C CNN
+F 3 "~" H 3450 2000 50  0001 C CNN
+	1    3450 2000
+	1    0    0    -1
+$EndComp
+Wire Wire Line
+	3600 1850 3450 1850
+Wire Wire Line
+	3450 1850 3300 1850
+Connection ~ 3450 1850
+Wire Wire Line
+	3300 1950 3300 2150
+Wire Wire Line
+	3300 2150 3450 2150
+$Comp
+L power:GND #PWR040
+U 1 1 5B663208
+P 3450 2150
+F 0 "#PWR040" H 3450 1900 50  0001 C CNN
+F 1 "GND" H 3455 1977 50  0000 C CNN
+F 2 "" H 3450 2150 50  0001 C CNN
+F 3 "" H 3450 2150 50  0001 C CNN
+	1    3450 2150
+	1    0    0    -1
+$EndComp
+Connection ~ 3450 2150
+$Comp
+L Connector:Conn_01x04_Male J?
+U 1 1 5B66F399
+P 4550 1350
+F 0 "J?" H 4523 1323 50  0000 R CNN
+F 1 "Conn_01x04_Male" H 4523 1232 50  0000 R CNN
+F 2 "" H 4550 1350 50  0001 C CNN
+F 3 "~" H 4550 1350 50  0001 C CNN
+	1    4550 1350
+	-1   0    0    -1
+$EndComp
+Wire Wire Line
+	3300 1250 4350 1250
+Wire Wire Line
+	4350 1350 3300 1350
+Wire Bus Line
+	1650 6400 10900 6400
+Wire Bus Line
+	9700 800  9700 2650
+Wire Bus Line
+	1600 4500 10350 4500
+$Comp
+L power:+3V3 #PWR?
+U 1 1 5B6822C7
+P 4350 1450
+F 0 "#PWR?" H 4350 1300 50  0001 C CNN
+F 1 "+3V3" H 4365 1623 50  0000 C CNN
+F 2 "" H 4350 1450 50  0001 C CNN
+F 3 "" H 4350 1450 50  0001 C CNN
+	1    4350 1450
+	0    -1   -1   0
+$EndComp
+$Comp
+L power:GND #PWR?
+U 1 1 5B68240D
+P 4350 1550
+F 0 "#PWR?" H 4350 1300 50  0001 C CNN
+F 1 "GND" H 4355 1377 50  0000 C CNN
+F 2 "" H 4350 1550 50  0001 C CNN
+F 3 "" H 4350 1550 50  0001 C CNN
+	1    4350 1550
+	1    0    0    -1
+$EndComp

Commit message: Schematic complete. PCB nearly done.
Parts:
- added C1, C10, C8, C9: 100n, Capacitor_SMD:C_1206_3216Metric_Pad1.42x1.75mm_HandSolder, symbol Device:C
- added D6, D7: 1N4763A 91V, Diode_SMD:D_MiniMELF_Handsoldering, symbol Device:D_Zener
- added Q21, Q22: MMBTA42, Package_TO_SOT_SMD:SOT-323_SC-70_Handsoldering, symbol Parts_Stash:MMBTA42
- added R40, R41: 33k, Resistor_SMD:R_0805_2012Metric_Pad1.15x1.40mm_HandSolder, symbol Device:R
- added R42, R43: 240k, Resistor_SMD:R_0805_2012Metric_Pad1.15x1.40mm_HandSolder, symbol Device:R
- added R44: 68R, Resistor_SMD:R_0805_2012Metric_Pad1.15x1.40mm_HandSolder, symbol Device:R
- added R45, R46: 15R, Resistor_SMD:R_0805_2012Metric_Pad1.15x1.40mm_HandSolder, symbol Device:R
- J4: renamed from J?; footprint (none) -> Connector_PinHeader_2.54mm:PinHeader_1x05_P2.54mm_Horizontal; symbol Connector:Conn_01x04_Male -> Connector:Conn_01x05_Male
- R38: footprint (none) -> OptoDevice:R_LDR_4.9x4.2mm_P2.54mm_Vertical
- RST1: renamed from SW1; footprint (none) -> Button_Switch_THT:SW_PUSH_6mm
- renumbered SW2 to FLASH1
Connections:
- net labels added: +5V, 180v, ANODE_N1, ANODE_N2, BLUE, CATHODE_N1, CATHODE_N2, DRIVE_BLUE, DRIVE_GREEN, DRIVE_LED_A1, DRIVE_LED_A2, DRIVE_LED_A3, DRIVE_LED_A4, DRIVE_RED, DRIVE_S1, DRIVE_S2, GREEN, RED
- net labels removed: +180V
- wire segments 179 -> 215
Other:
- moved on the sheet: U5

Commit message: First final draft ready (Ausf B)
Parts:
- added C11: 10uF, Capacitor_THT:CP_Radial_D5.0mm_P2.50mm, symbol Device:CP
- added C12: 22uF, Capacitor_THT:CP_Radial_D5.0mm_P2.50mm, symbol Device:CP
- added U7: THERMAL_VIA, PartsStash_RW:Thermal_Via, symbol Parts_Stash:THERMAL_VIA
Connections:
- wire segments 215 -> 220
Changed lines of the file:
@@
 $EndComp
 Wire Wire Line
-	6000 950  6200 950
+	6000 950  6050 950
 $Comp
 L power:+3V3 #PWR015
 U 1 1 5B5B5A7B
-P 6800 900
-F 0 "#PWR015" H 6800 750 50  0001 C CNN
-F 1 "+3V3" H 6815 1073 50  0000 C CNN
-F 2 "" H 6800 900 50  0001 C CNN
-F 3 "" H 6800 900 50  0001 C CNN
-	1    6800 900
+P 6900 900
+F 0 "#PWR015" H 6900 750 50  0001 C CNN
+F 1 "+3V3" H 6915 1073 50  0000 C CNN
+F 2 "" H 6900 900 50  0001 C CNN
+F 3 "" H 6900 900 50  0001 C CNN
+	1    6900 900
 	1    0    0    -1
 $EndComp
@@
 $EndComp
 Wire Wire Line
-	6800 950  6800 900
+	6800 950  6900 950
 Wire Wire Line
 	6500 1300 6500 1250
@@
 Wire Wire Line
 	6700 3450 6700 3400
+Connection ~ 6700 3400
+$Comp
+L Device:CP C11
+U 1 1 5B6D84E6
+P 6050 1100
+F 0 "C11" H 6168 1146 50  0000 L CNN
+F 1 "10uF" H 6168 1055 50  0000 L CNN
+F 2 "Capacitor_THT:CP_Radial_D5.0mm_P2.50mm" H 6088 950 50  0001 C CNN
+F 3 "~" H 6050 1100 50  0001 C CNN
+	1    6050 1100
+	1    0    0    -1
+$EndComp
+Connection ~ 6050 950
+Wire Wire Line
+	6050 950  6200 950
+$Comp
+L Device:CP C12
+U 1 1 5B6D89E2
+P 6900 1100
+F 0 "C12" H 7018 1146 50  0000 L CNN
+F 1 "22uF" H 7018 1055 50  0000 L CNN
+F 2 "Capacitor_THT:CP_Radial_D5.0mm_P2.50mm" H 6938 950 50  0001 C CNN
+F 3 "~" H 6900 1100 50  0001 C CNN
+	1    6900 1100
+	1    0    0    -1
+$EndComp
+Wire Wire Line
+	6900 950  6900 900
+Connection ~ 6900 950
+Wire Wire Line
+	6900 1250 6750 1250
+Connection ~ 6500 1250
+Wire Wire Line
+	6050 1250 6500 1250
 Wire Bus Line
 	7650 2850 10000 2850
@@
 Wire Bus Line
 	700  4500 11150 4500
-Connection ~ 6700 3400
+$Comp
+L Parts_Stash:THERMAL_VIA U7
+U 1 1 5B728D7F
+P 6750 1350
+F 0 "U7" H 6800 1400 50  0001 C CNN
+F 1 "THERMAL_VIA" H 6700 1650 50  0001 C CNN
+F 2 "PartsStash_RW:Thermal_Via" H 6600 1350 50  0001 C CNN
+F 3 "" H 6600 1350 50  0001 C CNN
+	1    6750 1350
+	-1   0    0    1
+$EndComp
+Connection ~ 6750 1250
+Wire Wire Line
+	6750 1250 6500 1250
 $EndSCHEMATC

Commit message: Nothing works now.
Parts:
- added U10, U11, U12, U13, U14, U15, U16, U8, U9: THERMAL_VIA, PartsStash_RW:Thermal_Via, symbol Parts_Stash:THERMAL_VIA
- FLASH1, RST1: footprint Button_Switch_THT:SW_PUSH_6mm -> Button_Switch_THT:SW_PUSH-12mm
- Q10, Q11, Q12, Q13, Q14, Q15, Q16, Q17, Q18, Q19, Q2, Q20, Q21, Q22, Q3, Q4, Q5, Q6, Q7, Q8, Q9: footprint Package_TO_SOT_SMD:SOT-323_SC-70_Handsoldering -> Package_TO_SOT_SMD:TSOT-23_HandSoldering
- U5: value AP1117-33 -> NCP1117-33G; footprint Package_TO_SOT_SMD:SOT-223-3_TabPin2 -> PartsStash_RW:DPACK2
Connections:
- wire segments 220 -> 227
