File: kicad/ausf_d/ausf_d.sch (KiCad schematic (older format))
At the start: 1 part

Commit message: Working version of ausf D is on the branch.
Parts:
- removed U?: ESP8266EX, Package_DFN_QFN:QFN-32-1EP_5x5mm_P0.5mm_EP3.45x3.45mm, symbol MCU_Espressif:ESP8266EX
- added C10: 22u, Capacitor_SMD:CP_Elec_6.3x5.8, symbol Device:CP
- added C9: 10u, Capacitor_SMD:CP_Elec_6.3x5.8, symbol Device:CP
- added J1: Jack-DC, PartsStash:AliExpress55mmBarrelJack, symbol Connector:Barrel_Jack_Switch
- added J3: Conn_02x10_Odd_Even, Connector_IDC:IDC-Header_2x08_P2.54mm_Vertical, symbol Connector_Generic:Conn_02x08_Odd_Even
- added Q3, Q4: BC847, Package_TO_SOT_SMD:SOT-23, symbol Transistor_BJT:BC847
- added R10, R9: 12k, Resistor_SMD:R_0805_2012Metric_Pad1.15x1.40mm_HandSolder, symbol Device:R
- added U3: ESP-12F, RF_Module:ESP-12E, symbol RF_Module:ESP-12F
- added U4: AMS1117CD-3.3, Package_TO_SOT_SMD:TO-252-3_TabPin2, symbol Regulator_Linear:AMS1117CD-3.3
Connections:
- net labels added: +3V3, +9V, +FILAMENT_DC, +HVDC, DTR, FILAMENT_CLK, GND, GPIO0, HSPI_CLK, HSPI_CS, HSPI_DATA, RST, RTS
- wire segments 0 -> 36

Commit message: Made version work with Ausf. A and Ausf. C
Parts:
- C10: footprint Capacitor_SMD:CP_Elec_6.3x5.8 -> Capacitor_Tantalum_SMD:CP_EIA-6032-28_Kemet-C_Pad2.25x2.35mm_HandSolder
- C9: footprint Capacitor_SMD:CP_Elec_6.3x5.8 -> Capacitor_Tantalum_SMD:CP_EIA-3528-12_Kemet-T_Pad1.50x2.35mm_HandSolder
Changed lines of the file:
@@
 F 0 "C10" H 5268 1596 50  0000 L CNN
 F 1 "22u" H 5268 1505 50  0000 L CNN
-F 2 "Capacitor_SMD:CP_Elec_6.3x5.8" H 5188 1400 50  0001 C CNN
+F 2 "Capacitor_Tantalum_SMD:CP_EIA-6032-28_Kemet-C_Pad2.25x2.35mm_HandSolder" H 5188 1400 50  0001 C CNN
 F 3 "~" H 5150 1550 50  0001 C CNN
 	1    5150 1550
@@
 F 0 "C9" H 4368 1596 50  0000 L CNN
 F 1 "10u" H 4368 1505 50  0000 L CNN
-F 2 "Capacitor_SMD:CP_Elec_6.3x5.8" H 4288 1400 50  0001 C CNN
+F 2 "Capacitor_Tantalum_SMD:CP_EIA-3528-12_Kemet-T_Pad1.50x2.35mm_HandSolder" H 4288 1400 50  0001 C CNN
 F 3 "~" H 4250 1550 50  0001 C CNN
 	1    4250 1550
