File: kicad/ausf_d/filament_psu.sch (KiCad schematic (older format))
At the start: 15 parts, among them J4 Conn_01x02, Q2 2SD669AD-C, T1 TRIM_EU-S64W, U2 MC34063AP

Commit message: Minor edits
Parts:
- Q2: symbol ausf_d-rescue:BD140G-esp-vfd-clock-eagle-import -> ausf_d-rescue:BD140G-esp-vfd-clock-eagle-import-ausf_d-rescue
- R4: symbol ausf_d-rescue:R-EU_0411_15-esp-vfd-clock-eagle-import -> ausf_d-rescue:R-EU_0411_15-esp-vfd-clock-eagle-import-ausf_d-rescue
- R5, R6, R7, R8: symbol ausf_d-rescue:R-EU_0204_7-esp-vfd-clock-eagle-import -> ausf_d-rescue:R-EU_0204_7-esp-vfd-clock-eagle-import-ausf_d-rescue
- U2: symbol ausf_d-rescue:MC34063AP-esp-vfd-clock-eagle-import -> ausf_d-rescue:MC34063AP-esp-vfd-clock-eagle-import-ausf_d-rescue
Changed lines of the file:
@@
 EESchema Schematic File Version 4
-LIBS:ausf_d-cache
-EELAYER 29 0
+EELAYER 30 0
 EELAYER END
 $Descr A4 11693 8268
@@
 	4950 5550 5100 5550
 $Comp
-L ausf_d-rescue:R-EU_0204_7-esp-vfd-clock-eagle-import R6
+L ausf_d-rescue:R-EU_0204_7-esp-vfd-clock-eagle-import-ausf_d-rescue R6
 U 1 1 5CD6CAB6
 P 4350 3450
@@
 $EndComp
 $Comp
-L ausf_d-rescue:R-EU_0204_7-esp-vfd-clock-eagle-import R5
+L ausf_d-rescue:R-EU_0204_7-esp-vfd-clock-eagle-import-ausf_d-rescue R5
 U 1 1 5CD6CABC
 P 4050 3150
@@
 $EndComp
 $Comp
-L ausf_d-rescue:R-EU_0411_15-esp-vfd-clock-eagle-import R4
+L ausf_d-rescue:R-EU_0411_15-esp-vfd-clock-eagle-import-ausf_d-rescue R4
 U 1 1 5CD6CAC2
 P 3750 4250
@@
 $EndComp
 $Comp
-L ausf_d-rescue:R-EU_0204_7-esp-vfd-clock-eagle-import R8
+L ausf_d-rescue:R-EU_0204_7-esp-vfd-clock-eagle-import-ausf_d-rescue R8
 U 1 1 5CD6CAC8
 P 4750 5550
@@
 $EndComp
 $Comp
-L ausf_d-rescue:R-EU_0204_7-esp-vfd-clock-eagle-import R7
+L ausf_d-rescue:R-EU_0204_7-esp-vfd-clock-eagle-import-ausf_d-rescue R7
 U 1 1 5CD6CACE
 P 4350 5850
@@
 $EndComp
 $Comp
-L ausf_d-rescue:BD140G-esp-vfd-clock-eagle-import Q2
+L ausf_d-rescue:BD140G-esp-vfd-clock-eagle-import-ausf_d-rescue Q2
 U 1 1 5CD6CAE0
 P 4350 2450
+AR Path="/5CD6CAE0" Ref="Q2"  Part="1"
+AR Path="/5CD5170D/5CD6CAE0" Ref="Q2"  Part="1"
 F 0 "Q2" H 3950 2750 59  0000 L BNN
 F 1 "2SD669AD-C" H 3950 2650 59  0000 L BNN
@@
 $EndComp
 $Comp
-L ausf_d-rescue:GND-esp-vfd-clock-eagle-import #U016
+L ausf_d-rescue:GND-esp-vfd-clock-eagle-import-ausf_d-rescue #U016
 U 1 1 5CD6CB0A
 P 6450 4250
@@
 	4950 2350 5500 2350
 $Comp
-L ausf_d-rescue:MC34063AP-esp-vfd-clock-eagle-import U2
+L ausf_d-rescue:MC34063AP-esp-vfd-clock-eagle-import-ausf_d-rescue U2
 U 1 1 5CD6CAB0
 P 5350 4250
