File: kicad/ausf_c/front_panel.sch (KiCad schematic (older format))
At the start: 12 parts, among them J2 Conn_01x26_Male, J3 Conn_01x26_Female, T1 IN-12, T2 IN-12, T3 IN-12, T4 IN-12

Commit message: PSU does not fit into the outline.
Parts:
- removed J2: Conn_01x26_Male, Connector_PinSocket_2.54mm:PinSocket_1x26_P2.54mm_Vertical, symbol Connector_Generic:Conn_01x26
- removed J3: Conn_01x26_Female, Connector_PinSocket_2.54mm:PinSocket_1x26_P2.54mm_Vertical, symbol Connector:Conn_01x26_Female
Connections:
- wire segments 206 -> 191
Changed lines of the file:
@@
 Wire Wire Line
 	8450 3850 10050 3850
-$Comp
-L Connector_Generic:Conn_01x26 J2
-U 1 1 5B3174A8
-P 2350 3650
-F 0 "J2" H 2456 5028 50  0000 C CNN
-F 1 "Conn_01x26_Male" H 2456 4937 50  0000 C CNN
-F 2 "Connector_PinSocket_2.54mm:PinSocket_1x26_P2.54mm_Vertical" H 2350 3650 50  0001 C CNN
-F 3 "~" H 2350 3650 50  0001 C CNN
-	1    2350 3650
-	-1   0    0    -1
-$EndComp
-Wire Wire Line
-	2550 2450 2800 2450
 Wire Wire Line
 	2800 2450 2800 1750
@@
 	2900 1650 2900 2550
 Wire Wire Line
-	2900 2550 2550 2550
-Wire Wire Line
-	2550 2650 3000 2650
-Wire Wire Line
 	3000 2650 3000 1550
 Wire Wire Line
@@
 Wire Wire Line
 	3100 1450 3100 2750
-Wire Wire Line
-	3100 2750 2550 2750
 $Comp
 L Parts_Stash:LED_RGB_CA D2
@@
 	3550 3250 3550 2850
 Wire Wire Line
-	3550 2850 2550 2850
-Wire Wire Line
 	3600 3950 2550 3950
 Wire Wire Line
@@
 Wire Wire Line
 	6700 5550 6700 6200
-$Comp
-L Connector:Conn_01x26_Female J3
-U 1 1 5B5EDBAE
-P 1900 3650
-F 0 "J3" H 1927 3626 50  0000 L CNN
-F 1 "Conn_01x26_Female" H 1927 3535 50  0000 L CNN
-F 2 "Connector_PinSocket_2.54mm:PinSocket_1x26_P2.54mm_Vertical" H 1900 3650 50  0001 C CNN
-F 3 "~" H 1900 3650 50  0001 C CNN
-	1    1900 3650
-	1    0    0    -1
-$EndComp
-Wire Wire Line
-	1700 2450 1500 2450
-Wire Wire Line
-	1700 2550 1500 2550
-Wire Wire Line
-	1700 2650 1500 2650
-Wire Wire Line
-	1700 2750 1500 2750
-Text HLabel 1500 2450 0    50   Input ~ 0
+Text HLabel 2350 2450 0    50   Input ~ 0
 ANODE_1
-Text HLabel 1500 2550 0    50   Input ~ 0
+Text HLabel 2350 2750 0    50   Input ~ 0
 ANODE_2
-Text HLabel 1500 2650 0    50   Input ~ 0
+Text HLabel 2350 2650 0    50   Input ~ 0
 ANODE_3
-Text HLabel 1500 2750 0    50   Input ~ 0
+Text HLabel 2350 2550 0    50   Input ~ 0
 ANODE_4
 Text Label 2650 2450 0    50   ~ 0
 A1
 Text Label 2650 2550 0    50   ~ 0
-A2
+A4
 Text Label 2650 2650 0    50   ~ 0
 A3
 Text Label 2650 2750 0    50   ~ 0
-A4
-Text HLabel 1500 3650 0    50   Input ~ 0
+A2
+Text HLabel 2350 3650 0    50   Input ~ 0
 DIGIT_0
-Text HLabel 1500 3350 0    50   Input ~ 0
+Text HLabel 2350 3350 0    50   Input ~ 0
 DIGIT_1
-Text HLabel 1500 3250 0    50   Input ~ 0
+Text HLabel 2350 3250 0    50   Input ~ 0
 DIGIT_2
-Text HLabel 1500 3150 0    50   Input ~ 0
+Text HLabel 2350 3150 0    50   Input ~ 0
 DIGIT_3
-Text HLabel 1500 2850 0    50   Input ~ 0
+Text HLabel 2350 2850 0    50   Input ~ 0
 DIGIT_4
-Text HLabel 1500 2950 0    50   Input ~ 0
+Text HLabel 2350 2950 0    50   Input ~ 0
 DIGIT_5
-Text HLabel 1500 3850 0    50   Input ~ 0
+Text HLabel 2350 3850 0    50   Input ~ 0
 DIGIT_6
-Text HLabel 1500 3550 0    50   Input ~ 0
+Text HLabel 2350 3550 0    50   Input ~ 0
 DIGIT_7
-Text HLabel 1500 3050 0    50   Input ~ 0
+Text HLabel 2350 3050 0    50   Input ~ 0
 DIGIT_8
-Text HLabel 1500 3750 0    50   Input ~ 0
+Text HLabel 2350 3750 0    50   Input ~ 0
 DIGIT_9
-Text HLabel 1500 3450 0    50   Input ~ 0
+Text HLabel 2350 3450 0    50   Input ~ 0
 DIGIT_DOT
-Wire Wire Line
-	1700 2850 1500 2850
-Wire Wire Line
-	1700 2950 1500 2950
-Wire Wire Line
-	1700 3050 1500 3050
-Wire Wire Line
-	1700 3150 1500 3150
-Wire Wire Line
-	1700 3250 1500 3250
-Wire Wire Line
-	1700 3350 1500 3350
-Wire Wire Line
-	1700 3450 1500 3450
-Wire Wire Line
-	1700 3550 1500 3550
-Wire Wire Line
-	1700 3650 1500 3650
-Wire Wire Line
-	1700 3750 1500 3750
-Wire Wire Line
-	1700 3850 1500 3850
 Wire Wire Line
 	3850 2650 3850 2750
@@
 Wire Wire Line
 	3450 3350 3450 2950
-Wire Wire Line
-	3450 2950 2550 2950
 Connection ~ 4150 3350
 Wire Wire Line
@@
 Wire Wire Line
 	3350 3650 3350 3050
-Wire Wire Line
-	3350 3050 2550 3050
 Connection ~ 4450 3650
 Wire Wire Line
@@
 Wire Wire Line
 	5850 3350 4150 3350
-Wire Wire Line
-	2550 3150 3950 3150
 Connection ~ 3950 3150
 Wire Wire Line
-	2550 3250 3250 3250
-Wire Wire Line
 	3250 3250 3250 2750
 Wire Wire Line
@@
 Wire Wire Line
 	3250 3450 3250 3350
-Wire Wire Line
-	3250 3350 2550 3350
 Connection ~ 3750 2950
-Wire Wire Line
-	2550 3450 3150 3450
 Wire Wire Line
 	3150 3450 3150 3850
@@
 	3150 3850 4650 3850
 Connection ~ 4650 3850
-Wire Wire Line
-	4350 3550 2550 3550
 Connection ~ 4350 3550
 Wire Wire Line
@@
 	3850 2750 3850 3050
 Wire Wire Line
-	2550 3650 3250 3650
-Wire Wire Line
 	3250 3650 3250 3700
 Wire Wire Line
@@
 	3650 3700 3650 2850
 Connection ~ 3650 2850
-Wire Wire Line
-	4550 3750 2550 3750
 Connection ~ 4550 3750
-Wire Wire Line
-	2550 3850 3100 3850
 Wire Wire Line
 	3100 3850 3100 3900
@@
 Text Label 2650 3850 0    50   ~ 0
 D6
-Text HLabel 1700 3950 0    50   Input ~ 0
+Text HLabel 2550 3950 0    50   Input ~ 0
 ANODE_N1
-Text HLabel 1700 4050 0    50   Input ~ 0
+Text HLabel 2550 4050 0    50   Input ~ 0
 CATHODE_N1
-Text HLabel 1700 4150 0    50   Input ~ 0
+Text HLabel 2550 4150 0    50   Input ~ 0
 ANODE_N2
-Text HLabel 1700 4250 0    50   Input ~ 0
+Text HLabel 2550 4250 0    50   Input ~ 0
 CATHODE_N2
-Text HLabel 1700 4350 0    50   Input ~ 0
+Text HLabel 2550 4350 0    50   Input ~ 0
 RED
-Text HLabel 1700 4450 0    50   Input ~ 0
+Text HLabel 2550 4450 0    50   Input ~ 0
 GREEN
-Text HLabel 1700 4550 0    50   Input ~ 0
+Text HLabel 2550 4550 0    50   Input ~ 0
 BLUE
-Text HLabel 1700 4650 0    50   Input ~ 0
+Text HLabel 2550 4650 0    50   Input ~ 0
 ANODE_LED_1
-Text HLabel 1700 4750 0    50   Input ~ 0
+Text HLabel 2550 4750 0    50   Input ~ 0
 ANODE_LED_2
-Text HLabel 1700 4850 0    50   Input ~ 0
+Text HLabel 2550 4850 0    50   Input ~ 0
 ANODE_LED_3
-Text HLabel 1700 4950 0    50   Input ~ 0
+Text HLabel 2550 4950 0    50   Input ~ 0
 ANODE_LED_4
+Wire Wire Line
+	2350 2450 2800 2450
+Wire Wire Line
+	2350 2550 2900 2550
+Wire Wire Line
+	2350 2650 3000 2650
+Wire Wire Line
+	2350 2750 3100 2750
+Wire Wire Line
+	2350 2850 3550 2850
+Wire Wire Line
+	2350 2950 3450 2950
+Wire Wire Line
+	2350 3050 3350 3050
+Wire Wire Line
+	2350 3150 3950 3150
+Wire Wire Line
+	2350 3250 3250 3250
+Wire Wire Line
+	2350 3350 3250 3350
+Wire Wire Line
+	2350 3450 3150 3450
+Wire Wire Line
+	2350 3550 4350 3550
+Wire Wire Line
+	2350 3650 3250 3650
+Wire Wire Line
+	2350 3750 4550 3750
+Wire Wire Line
+	2350 3850 3100 3850
 $EndSCHEMATC

Commit message: Nearly done Ausf C PCB layout.
Parts:
- D2, D3, D4, D5: symbol Parts_Stash:LED_RGB_CA -> funknetzwerkuhr-rescue:LED_RGB_CA-Parts_Stash
- L2, L3: symbol Russian_Lamps:ins-1 -> funknetzwerkuhr-rescue:ins-1-Russian_Lamps
- T1, T2, T3, T4: footprint Parts:IN-12_0.8mm -> PartsStash:IN-12_0.8mm_simple; symbol Russian_Lamps:IN-12 -> funknetzwerkuhr-rescue:IN-12-Russian_Lamps
Changed lines of the file:
@@
 EESchema Schematic File Version 4
 LIBS:funknetzwerkuhr-cache
-EELAYER 26 0
+EELAYER 29 0
 EELAYER END
 $Descr A4 11693 8268
@@
 $EndDescr
 $Comp
-L Russian_Lamps:IN-12 T1
+L funknetzwerkuhr-rescue:IN-12-Russian_Lamps T1
 U 1 1 5B30153D
 P 4150 2250
 F 0 "T1" V 4196 1522 50  0000 R CNN
 F 1 "IN-12" V 4105 1522 50  0000 R CNN
-F 2 "Parts:IN-12_0.8mm" H 4050 1950 50  0001 C CNN
+F 2 "PartsStash:IN-12_0.8mm_simple" H 4050 1950 50  0001 C CNN
 F 3 "" H 4050 1950 50  0001 C CNN
 	1    4150 2250
@@
 $EndComp
 $Comp
-L Russian_Lamps:IN-12 T2
+L funknetzwerkuhr-rescue:IN-12-Russian_Lamps T2
 U 1 1 5B3017C6
 P 5850 2250
 F 0 "T2" V 5896 1522 50  0000 R CNN
 F 1 "IN-12" V 5805 1522 50  0000 R CNN
-F 2 "Parts:IN-12_0.8mm" H 5750 1950 50  0001 C CNN
+F 2 "PartsStash:IN-12_0.8mm_simple" H 5750 1950 50  0001 C CNN
 F 3 "" H 5750 1950 50  0001 C CNN
 	1    5850 2250
@@
 $EndComp
 $Comp
-L Russian_Lamps:IN-12 T3
+L funknetzwerkuhr-rescue:IN-12-Russian_Lamps T3
 U 1 1 5B3018D2
 P 7950 2250
 F 0 "T3" V 7996 1522 50  0000 R CNN
 F 1 "IN-12" V 7905 1522 50  0000 R CNN
-F 2 "Parts:IN-12_0.8mm" H 7850 1950 50  0001 C CNN
+F 2 "PartsStash:IN-12_0.8mm_simple" H 7850 1950 50  0001 C CNN
 F 3 "" H 7850 1950 50  0001 C CNN
 	1    7950 2250
@@
 $EndComp
 $Comp
-L Russian_Lamps:IN-12 T4
+L funknetzwerkuhr-rescue:IN-12-Russian_Lamps T4
 U 1 1 5B301A1E
 P 9550 2250
 F 0 "T4" V 9596 1522 50  0000 R CNN
 F 1 "IN-12" V 9505 1522 50  0000 R CNN
-F 2 "Parts:IN-12_0.8mm" H 9450 1950 50  0001 C CNN
+F 2 "PartsStash:IN-12_0.8mm_simple" H 9450 1950 50  0001 C CNN
 F 3 "" H 9450 1950 50  0001 C CNN
 	1    9550 2250
@@
 	3100 1450 3100 2750
 $Comp
-L Parts_Stash:LED_RGB_CA D2
+L funknetzwerkuhr-rescue:LED_RGB_CA-Parts_Stash D2
 U 1 1 5B33640C
 P 4300 5500
+AR Path="/5B33640C" Ref="D2"  Part="1"
+AR Path="/5B5B1D70/5B33640C" Ref="D2"  Part="1"
 F 0 "D2" H 4300 5965 50  0000 C CNN
 F 1 "LED_RGB_CA" H 4300 5874 50  0000 C CNN
@@
 $EndComp
 $Comp
-L Parts_Stash:LED_RGB_CA D3
+L funknetzwerkuhr-rescue:LED_RGB_CA-Parts_Stash D3
 U 1 1 5B336836
 P 5800 5500
+AR Path="/5B336836" Ref="D3"  Part="1"
+AR Path="/5B5B1D70/5B336836" Ref="D3"  Part="1"
 F 0 "D3" H 5800 5965 50  0000 C CNN
 F 1 "LED_RGB_CA" H 5800 5874 50  0000 C CNN
@@
 $EndComp
 $Comp
-L Parts_Stash:LED_RGB_CA D4
+L funknetzwerkuhr-rescue:LED_RGB_CA-Parts_Stash D4
 U 1 1 5B336AC2
 P 7900 5500
+AR Path="/5B336AC2" Ref="D4"  Part="1"
+AR Path="/5B5B1D70/5B336AC2" Ref="D4"  Part="1"
 F 0 "D4" H 7900 5965 50  0000 C CNN
 F 1 "LED_RGB_CA" H 7900 5874 50  0000 C CNN
@@
 $EndComp
 $Comp
-L Parts_Stash:LED_RGB_CA D5
+L funknetzwerkuhr-rescue:LED_RGB_CA-Parts_Stash D5
 U 1 1 5B336BFA
 P 9400 5500
+AR Path="/5B336BFA" Ref="D5"  Part="1"
+AR Path="/5B5B1D70/5B336BFA" Ref="D5"  Part="1"
 F 0 "D5" H 9400 5965 50  0000 C CNN
 F 1 "LED_RGB_CA" H 9400 5874 50  0000 C CNN
@@
 	8800 4450 8800 5650
 $Comp
-L Russian_Lamps:ins-1 L2
+L funknetzwerkuhr-rescue:ins-1-Russian_Lamps L2
 U 1 1 5B36A59C
 P 6800 5100
@@
 $EndComp
 $Comp
-L Russian_Lamps:ins-1 L3
+L funknetzwerkuhr-rescue:ins-1-Russian_Lamps L3
 U 1 1 5B36A720
 P 6800 5400

Commit message: Opened ausf_c with newer Kicad version.
Parts:
- D2, D3, D4, D5: symbol funknetzwerkuhr-rescue:LED_RGB_CA-Parts_Stash -> funknetzwerkuhr-rescue:LED_RGB_CA-Parts_Stash-funknetzwerkuhr-rescue
- L2, L3: symbol funknetzwerkuhr-rescue:ins-1-Russian_Lamps -> funknetzwerkuhr-rescue:ins-1-Russian_Lamps-funknetzwerkuhr-rescue
- T1, T2, T3, T4: symbol funknetzwerkuhr-rescue:IN-12-Russian_Lamps -> funknetzwerkuhr-rescue:IN-12-Russian_Lamps-funknetzwerkuhr-rescue
Changed lines of the file:
@@
 EESchema Schematic File Version 4
-LIBS:funknetzwerkuhr-cache
-EELAYER 29 0
+EELAYER 30 0
 EELAYER END
 $Descr A4 11693 8268
@@
 $EndDescr
 $Comp
-L funknetzwerkuhr-rescue:IN-12-Russian_Lamps T1
+L funknetzwerkuhr-rescue:IN-12-Russian_Lamps-funknetzwerkuhr-rescue T1
 U 1 1 5B30153D
 P 4150 2250
@@
 $EndComp
 $Comp
-L funknetzwerkuhr-rescue:IN-12-Russian_Lamps T2
+L funknetzwerkuhr-rescue:IN-12-Russian_Lamps-funknetzwerkuhr-rescue T2
 U 1 1 5B3017C6
 P 5850 2250
@@
 $EndComp
 $Comp
-L funknetzwerkuhr-rescue:IN-12-Russian_Lamps T3
+L funknetzwerkuhr-rescue:IN-12-Russian_Lamps-funknetzwerkuhr-rescue T3
 U 1 1 5B3018D2
 P 7950 2250
@@
 $EndComp
 $Comp
-L funknetzwerkuhr-rescue:IN-12-Russian_Lamps T4
+L funknetzwerkuhr-rescue:IN-12-Russian_Lamps-funknetzwerkuhr-rescue T4
 U 1 1 5B301A1E
 P 9550 2250
@@
 	3100 1450 3100 2750
 $Comp
-L funknetzwerkuhr-rescue:LED_RGB_CA-Parts_Stash D2
+L funknetzwerkuhr-rescue:LED_RGB_CA-Parts_Stash-funknetzwerkuhr-rescue D2
 U 1 1 5B33640C
 P 4300 5500
@@
 $EndComp
 $Comp
-L funknetzwerkuhr-rescue:LED_RGB_CA-Parts_Stash D3
+L funknetzwerkuhr-rescue:LED_RGB_CA-Parts_Stash-funknetzwerkuhr-rescue D3
 U 1 1 5B336836
 P 5800 5500
@@
 $EndComp
 $Comp
-L funknetzwerkuhr-rescue:LED_RGB_CA-Parts_Stash D4
+L funknetzwerkuhr-rescue:LED_RGB_CA-Parts_Stash-funknetzwerkuhr-rescue D4
 U 1 1 5B336AC2
 P 7900 5500
@@
 $EndComp
 $Comp
-L funknetzwerkuhr-rescue:LED_RGB_CA-Parts_Stash D5
+L funknetzwerkuhr-rescue:LED_RGB_CA-Parts_Stash-funknetzwerkuhr-rescue D5
 U 1 1 5B336BFA
 P 9400 5500
@@
 	8800 4450 8800 5650
 $Comp
-L funknetzwerkuhr-rescue:ins-1-Russian_Lamps L2
+L funknetzwerkuhr-rescue:ins-1-Russian_Lamps-funknetzwerkuhr-rescue L2
 U 1 1 5B36A59C
 P 6800 5100
@@
 $EndComp
 $Comp
-L funknetzwerkuhr-rescue:ins-1-Russian_Lamps L3
+L funknetzwerkuhr-rescue:ins-1-Russian_Lamps-funknetzwerkuhr-rescue L3
 U 1 1 5B36A720
 P 6800 5400
