File: kicad/ausf_c/hv_psu.sch (KiCad schematic (older format))
At the start: 17 parts, among them J1 Jack-DC, Q1 IRF640, U4 max1771

Commit message: PSU does not fit into the outline.
Parts:
- removed C13: 10uF,25V, Capacitor_THT:CP_Radial_D5.0mm_P2.50mm, symbol Device:CP
- removed C6: 100p 1kV, Capacitor_THT:C_Disc_D6.0mm_W2.5mm_P5.00mm, symbol Device:C
- C4: footprint Capacitor_THT:CP_Radial_D8.0mm_P3.50mm -> Capacitor_SMD:CP_Elec_8x10.5
- D1: footprint Parts:D_MELF-RM10_Universal_Handsoldering -> Diode_SMD:D_SMB_Handsoldering
- L1: footprint PartsStash_RW:L_Toroid_Horizontal_D16.8mm_P6mm_AliExpress -> Inductor_THT:L_Toroid_Vertical_L14.0mm_W6.3mm_P4.57mm_Pulse_A
- RSENSE1: footprint Resistor_THT:R_Axial_DIN0414_L11.9mm_D4.5mm_P15.24mm_Horizontal -> Resistor_SMD:R_2512_6332Metric_Pad1.52x3.35mm_HandSolder
Connections:
- net labels added: SENSE
- wire segments 63 -> 56
Changed lines of the file:
@@
 F 0 "L1" V 6440 2700 50  0000 C CNN
 F 1 "L" V 6349 2700 50  0000 C CNN
-F 2 "PartsStash_RW:L_Toroid_Horizontal_D16.8mm_P6mm_AliExpress" H 6250 2700 50  0001 C CNN
+F 2 "Inductor_THT:L_Toroid_Vertical_L14.0mm_W6.3mm_P4.57mm_Pulse_A" H 6250 2700 50  0001 C CNN
 F 3 "" H 6250 2700 50  0001 C CNN
 	1    6250 2700
@@
 L Device:CP C4
 U 1 1 5B7B059A
-P 5900 2850
-F 0 "C4" V 6000 2700 50  0000 L CNN
-F 1 "100uF,25V" V 5750 2700 50  0000 L CNN
-F 2 "Capacitor_THT:CP_Radial_D8.0mm_P3.50mm" H 5938 2700 50  0001 C CNN
-F 3 "" H 5900 2850 50  0001 C CNN
-	1    5900 2850
+P 3900 3500
+F 0 "C4" V 4000 3350 50  0000 L CNN
+F 1 "100uF,25V" V 3750 3350 50  0000 L CNN
+F 2 "Capacitor_SMD:CP_Elec_8x10.5" H 3938 3350 50  0001 C CNN
+F 3 "" H 3900 3500 50  0001 C CNN
+	1    3900 3500
 	1    0    0    -1
 $EndComp
@@
 F 0 "RSENSE1" V 6500 4200 50  0000 L CNN
 F 1 "0R1" V 6700 4200 50  0000 L CNN
-F 2 "Resistor_THT:R_Axial_DIN0414_L11.9mm_D4.5mm_P15.24mm_Horizontal" V 6530 4300 50  0001 C CNN
+F 2 "Resistor_SMD:R_2512_6332Metric_Pad1.52x3.35mm_HandSolder" V 6530 4300 50  0001 C CNN
 F 3 "" H 6600 4300 50  0001 C CNN
 	1    6600 4300
@@
 F 0 "D1" H 6950 2484 50  0000 C CNN
 F 1 "ES2J" H 6950 2575 50  0000 C CNN
-F 2 "Parts:D_MELF-RM10_Universal_Handsoldering" H 6950 2700 50  0001 C CNN
+F 2 "Diode_SMD:D_SMB_Handsoldering" H 6950 2700 50  0001 C CNN
 F 3 "" H 6950 2700 50  0001 C CNN
 	1    6950 2700
@@
 Connection ~ 7300 4550
 Wire Wire Line
-	7700 2950 7700 2850
-Wire Wire Line
 	7700 2700 7300 2700
 Connection ~ 7300 2700
@@
 Wire Wire Line
 	6950 3600 7700 3600
-Wire Wire Line
-	7700 3600 7700 3350
 $Comp
 L Device:C C7
@@
 Wire Wire Line
 	7700 4150 7700 4050
-$Comp
-L Device:C C6
-U 1 1 5B5BDFDB
-P 8050 3100
-F 0 "C6" H 8165 3146 50  0000 L CNN
-F 1 "100p 1kV" H 8165 3055 50  0000 L CNN
-F 2 "Capacitor_THT:C_Disc_D6.0mm_W2.5mm_P5.00mm" H 8088 2950 50  0001 C CNN
-F 3 "~" H 8050 3100 50  0001 C CNN
-	1    8050 3100
-	1    0    0    -1
-$EndComp
-Wire Wire Line
-	8050 2950 8050 2850
-Wire Wire Line
-	8050 2850 7700 2850
-Connection ~ 7700 2850
-Wire Wire Line
-	7700 2850 7700 2700
-Wire Wire Line
-	8050 3250 8050 3350
-Wire Wire Line
-	8050 3350 7700 3350
-Connection ~ 7700 3350
-Wire Wire Line
-	7700 3350 7700 3250
 Text HLabel 8800 2700 2    50   Output ~ 0
 +180V
@@
 Wire Wire Line
 	3900 4550 3500 4550
-Wire Wire Line
-	5550 2700 5900 2700
 Wire Wire Line
 	3900 3350 3900 2700
@@
 	0    1    1    0
 $EndComp
-Connection ~ 5900 2700
-Wire Wire Line
-	5900 2700 6100 2700
-$Comp
-L power:GND #PWR049
-U 1 1 5B7288C4
-P 5900 3000
-F 0 "#PWR049" H 5900 2750 50  0001 C CNN
-F 1 "GND" H 5905 2827 50  0000 C CNN
-F 2 "" H 5900 3000 50  0001 C CNN
-F 3 "" H 5900 3000 50  0001 C CNN
-	1    5900 3000
-	1    0    0    -1
-$EndComp
-$Comp
-L Device:CP C13
-U 1 1 5B7288EF
-P 3900 3500
-F 0 "C13" V 4000 3350 50  0000 L CNN
-F 1 "10uF,25V" V 3750 3350 50  0000 L CNN
-F 2 "Capacitor_THT:CP_Radial_D5.0mm_P2.50mm" H 3938 3350 50  0001 C CNN
-F 3 "" H 3900 3500 50  0001 C CNN
-	1    3900 3500
-	1    0    0    -1
-$EndComp
+Wire Wire Line
+	7700 2700 7700 2950
+Wire Wire Line
+	7700 3250 7700 3600
+Wire Wire Line
+	5550 2700 6100 2700
+Text Label 6600 3900 3    50   ~ 0
+SENSE
 $EndSCHEMATC

Commit message: Nearly done Ausf C PCB layout.
Parts:
- R1a1, R2, R34: footprint Resistor_SMD:R_0805_2012Metric_Pad1.15x1.40mm_HandSolder -> PartsStash:R_0805_2012Metric_Pad1.15x1.40mm_HandSolder_Value
- U4: symbol Parts_Stash:MAX1771 -> funknetzwerkuhr-rescue:MAX1771-Parts_Stash
Changed lines of the file:
@@
 EESchema Schematic File Version 4
 LIBS:funknetzwerkuhr-cache
-EELAYER 26 0
+EELAYER 29 0
 EELAYER END
 $Descr A4 11693 8268
@@
 	4100 2050 4100 1950
 $Comp
-L Parts_Stash:MAX1771 U4
+L funknetzwerkuhr-rescue:MAX1771-Parts_Stash U4
 U 1 1 5B71C581
 P 5550 3800
+AR Path="/5B71C581" Ref="U4"  Part="1"
+AR Path="/5B5B1780/5B71C581" Ref="U4"  Part="1"
 F 0 "U4" H 5250 4250 50  0000 C CNN
 F 1 "max1771" H 5300 3400 50  0000 C CNN
@@
 F 0 "R2" H 7770 4346 50  0000 L CNN
 F 1 "10k" H 7770 4255 50  0000 L CNN
-F 2 "Resistor_SMD:R_0805_2012Metric_Pad1.15x1.40mm_HandSolder" V 7630 4300 50  0001 C CNN
+F 2 "PartsStash:R_0805_2012Metric_Pad1.15x1.40mm_HandSolder_Value" V 7630 4300 50  0001 C CNN
 F 3 "" H 7700 4300 50  0001 C CNN
 	1    7700 4300
@@
 F 0 "R1a1" H 7770 3946 50  0000 L CNN
 F 1 "2.7k" H 7770 3855 50  0000 L CNN
-F 2 "Resistor_SMD:R_0805_2012Metric_Pad1.15x1.40mm_HandSolder" V 7630 3900 50  0001 C CNN
+F 2 "PartsStash:R_0805_2012Metric_Pad1.15x1.40mm_HandSolder_Value" V 7630 3900 50  0001 C CNN
 F 3 "" H 7700 3900 50  0001 C CNN
 	1    7700 3900
@@
 F 0 "R34" V 4743 3600 50  0000 C CNN
 F 1 "0R0" V 4834 3600 50  0000 C CNN
-F 2 "Resistor_SMD:R_0805_2012Metric_Pad1.15x1.40mm_HandSolder" V 4880 3600 50  0001 C CNN
+F 2 "PartsStash:R_0805_2012Metric_Pad1.15x1.40mm_HandSolder_Value" V 4880 3600 50  0001 C CNN
 F 3 "~" H 4950 3600 50  0001 C CNN
 	1    4950 3600

Commit message: Ausf C PCB version ordered.
Parts:
- added J3: Conn_01x02_Male, Connector_PinHeader_2.54mm:PinHeader_1x02_P2.54mm_Vertical, symbol Connector:Conn_01x02_Male
- C4: value 100uF,25V -> 220uF,25V; footprint Capacitor_SMD:CP_Elec_8x10.5 -> Capacitor_THT:CP_Radial_D10.0mm_P2.50mm_P5.00mm
Connections:
- net +VDC: now also J3.2 (Pin_2)
- net GND: now also J3.1 (Pin_1)
Changed lines of the file:
@@
 	0    -1   -1   0
-$EndComp
-$Comp
-L Device:CP C4
-U 1 1 5B7B059A
-P 3900 3500
-F 0 "C4" V 4000 3350 50  0000 L CNN
-F 1 "100uF,25V" V 3750 3350 50  0000 L CNN
-F 2 "Capacitor_SMD:CP_Elec_8x10.5" H 3938 3350 50  0001 C CNN
-F 3 "" H 3900 3500 50  0001 C CNN
-	1    3900 3500
-	1    0    0    -1
 $EndComp
 Wire Wire Line
@@
 $EndComp
 Wire Wire Line
-	8550 2700 8550 3450
+	8550 2700 8550 3000
 Wire Wire Line
 	7700 2700 8550 2700
@@
 Text Label 6600 3900 3    50   ~ 0
 SENSE
+$Comp
+L Device:CP C4
+U 1 1 5B7B059A
+P 3900 3500
+F 0 "C4" V 4000 3350 50  0000 L CNN
+F 1 "220uF,25V" V 3750 3350 50  0000 L CNN
+F 2 "Capacitor_THT:CP_Radial_D10.0mm_P2.50mm_P5.00mm" H 3938 3350 50  0001 C CNN
+F 3 "" H 3900 3500 50  0001 C CNN
+	1    3900 3500
+	1    0    0    -1
+$EndComp
+$Comp
+L Connector:Conn_01x02_Male J3
+U 1 1 5CCD2A7A
+P 9150 3100
+F 0 "J3" H 9122 2982 50  0000 R CNN
+F 1 "Conn_01x02_Male" H 9122 3073 50  0000 R CNN
+F 2 "Connector_PinHeader_2.54mm:PinHeader_1x02_P2.54mm_Vertical" H 9150 3100 50  0001 C CNN
+F 3 "~" H 9150 3100 50  0001 C CNN
+	1    9150 3100
+	-1   0    0    1
+$EndComp
+Wire Wire Line
+	8550 3000 8950 3000
+Connection ~ 8550 3000
+Wire Wire Line
+	8550 3000 8550 3450
+Wire Wire Line
+	8950 3100 8950 4550
+Wire Wire Line
+	8950 4550 8550 4550
+Connection ~ 8550 4550
 $EndSCHEMATC

Commit message: Opened ausf_c with newer Kicad version.
Parts:
- U4: symbol funknetzwerkuhr-rescue:MAX1771-Parts_Stash -> funknetzwerkuhr-rescue:MAX1771-Parts_Stash-funknetzwerkuhr-rescue
Changed lines of the file:
@@
 EESchema Schematic File Version 4
-LIBS:funknetzwerkuhr-cache
-EELAYER 29 0
+EELAYER 30 0
 EELAYER END
 $Descr A4 11693 8268
@@
 	4100 2050 4100 1950
 $Comp
-L funknetzwerkuhr-rescue:MAX1771-Parts_Stash U4
+L funknetzwerkuhr-rescue:MAX1771-Parts_Stash-funknetzwerkuhr-rescue U4
 U 1 1 5B71C581
 P 5550 3800
