File: kicad/ausf_c/funknetzwerkuhr.kicad_pcb (KiCad board)
At the start: 2 copper layers, 100 x 80 mm, 110 parts, among them J1 Jack-DC, J2 Conn_01x04_Male, J3 180V, J4 Conn_01x04_Male, Q1 IRF640, Q10 MMBTA42, Q11 MMBTA42, Q12 MMBTA42, Q13 MMBTA42, Q14 MMBTA42, Q15 MMBTA42, Q16 MMBTA42, Q17 MMBTA42, Q18 MMBTA42, Q19 MMBTA42, Q2 MMBTA42, Q20 MMBTA42, Q21 MMBTA42, Q22 MMBTA42, Q3 MMBTA92, Q4 MMBTA42, Q5 MMBTA92, Q6 MMBTA42, Q7 MMBTA92, Q8 MMBTA42, Q9 MMBTA92, T1 IN-12, T2 IN-12, T3 IN-12, T4 IN-12, U1 74HC595, U2 74HC595, U3 74HC595, U4 max1771, U5 NCP1117-33G, U6 ESP-12E

Commit message: Opened ausf_c with newer Kicad version.
Parts:
- J3: value 180V -> Conn_01x02_Male

Commit message: Added Ausf C layout
Connections:
- net /~OE renamed /~{OE}
Other:
- net class Default removed
- net class Power removed
